File: FlightComputer.kicad_pcb (KiCad board)
At the start: 4 copper layers, 83 x 62 mm, 153 parts, among them IC1 LMR33640DDDAR, J1 SM05B-GHS-TB, J10 Header1x3Pin, J11 Header1x3Pin, J12 Header1x3Pin, J13 SM02B-GHS-TB, J14 Header1x3Pin, J15 Header1x3Pin, J16 Header1x3Pin, J17 SM02B-GHS-TB, J18 USB_C_Receptacle, J19 SM02B-GHS-TB, J2 Screw_Terminal_01x02, J3 SM07B-GHS-TB, J4 SM05B-GHS-TB, J5 SM07B-GHS-TB, J6 SM05B-GHS-TB, J7 SM07B-GHS-TB, J8 SM05B-GHS-TB, J9 SM05B-GHS-TB, Q1 SI2369BDS-T1-GE3 30V 5.6A, SW1 KMR221GLFS, SW2 KMR221GLFS, U1 LIS3MDL, U2 BMI270, U3 AP7361C-33ER-13, U4 STM32F446RET6, U5 LPS22HH, U6 NEO-M9N, U7 W25Q128JVSIQ, Y1 16MHz

Commit message: Add files via upload
Parts:
- removed D10, D11, D12, D13, D14, D15, D16, D17, D18, D19, D20, D21, D22, D23, D24, D25, D26, D27, D28, D29, D30, D31, D38, D39, D40, D41, D42, D43, D5, D6, D7, D8, D9: CESD3V3D3 YU, Diode_SMD:D_SOD-323
- removed D33, D34: PESD3V3U1UA,115, Diode_SMD:D_SOD-323
- added U10: USBLC6-4SC6, Package_TO_SOT_SMD:SOT-23-6, F.Cu at (96.6, 66.3)
- added U11: USBLC6-4SC6, Package_TO_SOT_SMD:SOT-23-6, F.Cu at (108.2, 66.2)
- added U12: USBLC6-4SC6, Package_TO_SOT_SMD:SOT-23-6, F.Cu at (121.5, 100.7)
- added U13: USBLC6-4SC6, Package_TO_SOT_SMD:SOT-23-6, F.Cu at (121.5, 105.9)
- added U14: USBLC6-4SC6, Package_TO_SOT_SMD:SOT-23-6, F.Cu at (116.5, 110.5)
- added U15: USBLC6-4SC6, Package_TO_SOT_SMD:SOT-23-6, F.Cu at (111.8, 110.5)
- added U16: USBLC6-4SC6, Package_TO_SOT_SMD:SOT-23-6, F.Cu at (94.0, 110.7)
- added U17: USBLC6-4SC6, Package_TO_SOT_SMD:SOT-23-6, F.Cu at (89.5, 110.8)
- added U18: USBLC6-4SC6, Package_TO_SOT_SMD:SOT-23-6, F.Cu at (79.8, 110.6)
- added U19: USBLC6-4SC6, Package_TO_SOT_SMD:SOT-23-6, F.Cu at (57.9, 87.5)
- added U20: USBLC6-4SC6, Package_TO_SOT_SMD:SOT-23-6, F.Cu at (122.2, 88.1)
- added U8: USBLC6-4SC6, Package_TO_SOT_SMD:SOT-23-6, F.Cu at (73.7, 66.3)
- added U9: USBLC6-4SC6, Package_TO_SOT_SMD:SOT-23-6, F.Cu at (85.2, 66.3)
- D3, D32, D4: value CESD3V3D3 YU -> PESD5V0U1UA
- D36: value CESD5V0D1-ES -> PESD5V0U1UA
- moved D3 72.9 mm to (57.8, 72.9), turned to 0 degrees
- moved D4 68.7 mm to (57.8, 80.9), turned to 0 degrees
- moved F6 2.92 mm to (119.3, 110.6)
- moved C3 2.45 mm to (74.2, 74.1), turned to 90 degrees
- moved J1 2.41 mm to (108.2, 60.8)
- moved F3 2.33 mm to (93.6, 66.3)
- moved F7 1.97 mm to (56.9, 91.1), turned to -90 degrees
- moved F2 1.77 mm to (82.3, 66.3)
- moved C1 1.57 mm to (74.2, 77.1), turned to -90 degrees
- moved J8 1.55 mm to (96.7, 60.8)
- moved F1 0.86 mm to (70.8, 66.2)
- moved J6 0.80 mm to (85.2, 60.8)
- moved F4 0.74 mm to (82.7, 110.8)
- moved D1 0.60 mm to (90.8, 102.1)
- moved R9 0.60 mm to (92.8, 102.1)
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Connections:
- D3 pad 1: Servo 1 -> Net-(D3-K)
- D4 pad 1: Servo 2 -> Net-(D4-K)
- F7 pad 1: Net-(J5-Pin_1) -> Net-(J5-Pin_3)
- F8 pad 2: Net-(J17-Pin_1) -> Net-(D4-K)
- F9 pad 2: Net-(J13-Pin_1) -> Net-(D3-K)
- J1 pad 1: NRST -> SWO
- J1 pad 2: SWO -> NRST
- J1 pad 4: SWCLK -> SWDIO
- J1 pad 5: SWDIO -> SWCLK
- J13 pad 1: Net-(J13-Pin_1) -> Net-(D3-K)
- J17 pad 1: Net-(J17-Pin_1) -> Net-(D4-K)
- J3 pad 3: CE -> GND
- J3 pad 4: GND -> CE
- J5 pad 1: Net-(J5-Pin_1) -> GND
- J5 pad 2: Net-(J5-Pin_1) -> GND
- J5 pad 3: GND -> Net-(J5-Pin_3)
- J5 pad 4: GND -> Net-(J5-Pin_3)
- U4 pad 10: unconnected-(U4-PC2-Pad10) -> INT5
- U4 pad 11: unconnected-(U4-PC3-Pad11) -> INT4
- U4 pad 2: unconnected-(U4-PC13-Pad2) -> INT1
- U4 pad 4: unconnected-(U4-PC15-Pad4) -> INT2
- U4 pad 54: unconnected-(U4-PD2-Pad54) -> INT3
Routing:
- net GND: track 13.2 -> 65.8 mm, vias 271 -> 294
- net INT1: track 0.00 -> 41.3 mm, vias 0 -> 2
- net INT5: track 0.00 -> 34.9 mm, vias 0 -> 2
- net INT2: track 0.00 -> 33.0 mm, vias 0 -> 2
- net INT4: track 2.47 -> 33.4 mm, vias 0 -> 2
- net INT3: track 0.00 -> 28.4 mm, vias 0 -> 2
- net SCL: track 79.8 -> 99.6 mm, vias 4 -> 7
- net NRST: track 38.6 -> 49.3 mm
- net Servo 1: track 31.1 -> 41.3 mm
- net SWDIO: track 26.6 -> 35.9 mm
- net Net-(J4-Pin_1): track 0.00 -> 4.98 mm
- net +3V3: track 35.2 -> 30.9 mm
- net SWCLK: track 22.0 -> 25.8 mm
- net Servo 2: track 26.1 -> 29.8 mm, vias 0 -> 1
- net SCK: track 54.0 -> 57.6 mm, vias 2 -> 3
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- added copper zone on F.Cu, net Net-(D3-K)
- added copper zone on F.Cu, net Net-(D4-K)
- added copper zone on F.Cu, net Net-(J5-Pin_3)
- removed copper zone on F.Cu, net Net-(J5-Pin_1)
Other:
- board text added: "3V3 CS SCK MOSI MISO INT GND"
- board text added: "3V3 CSN GND CS MOSI SCK MISO"
- board text added: "3V3 INT RX TX GND"
- board text added: "GND INT SDA SCL 3V3"
- board text removed: "3V3 CS SCK MOSI MISO GND"
- board text removed: "3V3 CSN CS GND MOSI SCK MISO"
- board text removed: "3V3 RX TX GND"
- board text removed: "GND SDA SCL 3V3"

Commit message: Add files via upload
Parts:
- moved U19 0.45 mm to (57.9, 87.0)
- moved F7 0.45 mm to (56.9, 90.7)
- moved J5 0.45 mm to (52.8, 89.4)
- moved U20 0.25 mm to (122.5, 88.1)
- moved F8 0.20 mm to (56.9, 78.3)
- moved J17 0.20 mm to (52.8, 78.5)
- moved D4 0.10 mm to (57.8, 80.8)
- moved D3 0.10 mm to (57.8, 73.0)
Routing:
- net Servo 1: track 41.3 -> 34.8 mm
- net GND: track 65.8 -> 65.3 mm, vias 294 -> 293
Other:
- board text removed: "5V OUT"

Commit message: Add files via upload
Parts:
- moved U3 0.40 mm to (62.4, 65.4)
- moved C26 0.40 mm to (57.2, 65.4)
- moved C27 0.40 mm to (62.5, 60.9)
- moved J1 0.10 mm to (108.1, 60.8)
- moved U11 0.10 mm to (108.1, 66.2)
- renumbered D32 to D5
Routing:
- net GND: track 65.3 -> 66.8 mm, vias 293 -> 297
Other:
- board text added: "SWCLK SWDIO GND MRST SWO"
- board text added: "TX RX INT 5V 5V GND GND"
- board text removed: "SWDIO SWCLK GND SWO NRST"
- board text removed: "TX RX INT GND GND 5V 5V"

Commit message: Add files via upload
Changed lines of the file:
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@@
     (property "ki_keywords" "usb ethernet sim card video")
     (attr smd)
-    (fp_text reference "U17" (at -0.0125 -2.6) (layer "F.SilkS")
+    (fp_text reference "U17" (at -0.0125 -2.65) (layer "F.SilkS")
         (effects (font (size 1 1) (thickness 0.15)))
     )
@@
     (property "ki_keywords" "fuse")
     (attr smd)
-    (fp_text reference "F4" (at 2.8125 0.05 90) (layer "F.SilkS")
+    (fp_text reference "F4" (at 2.8125 0.03125 90) (layer "F.SilkS")
         (effects (font (size 1 1) (thickness 0.15)))
     )
@@
     (property "ki_keywords" "R res resistor")
     (attr smd)
-    (fp_text reference "R14" (at 3.275 0) (layer "F.SilkS")
+    (fp_text reference "R14" (at 3.1 0) (layer "F.SilkS")
         (effects (font (size 1 1) (thickness 0.15)))
     )
@@
     (property "ki_keywords" "R res resistor")
     (attr smd)
-    (fp_text reference "R13" (at 3.275 0) (layer "F.SilkS")
+    (fp_text reference "R13" (at 3.1 0) (layer "F.SilkS")
         (effects (font (size 1 1) (thickness 0.15)))
     )
@@
     (effects (font (size 1 1) (thickness 0.15)))
   )
-  (gr_text "I2C" (at 88.45 70.2) (layer "F.SilkS")
+  (gr_text "I2C" (at 78.85 66.2) (layer "F.SilkS")
     (effects (font (size 1 1) (thickness 0.15)))
   )
@@
   (segment (start 85.275 67.598528) (end 84.773528 68.1) (width 0.5) (layer "F.Cu") (net 6))
   (segment (start 109.194607 66.25) (end 108.633579 66.25) (width 0.5) (layer "F.Cu") (net 6))
+  (segment (start 79.8375 109.251472) (end 79.8375 109.998528) (width 0.5) (layer "F.Cu") (net 6))
   (segment (start 119.55 100.675) (end 120.848528 100.675) (width 0.5) (layer "F.Cu") (net 6))
   (segment (start 89.45 110.2) (end 89.45 108.9) (width 0.5) (layer "F.Cu") (net 6))
@@
   (segment (start 115.873528 110.55) (end 115.3125 110.55) (width 0.5) (layer "F.Cu") (net 6))
   (segment (start 108.057107 65.673528) (end 108.057107 64.2) (width 0.5) (layer "F.Cu") (net 6))
+  (segment (start 80.488972 108.6) (end 79.8375 109.251472) (width 0.5) (layer "F.Cu") (net 6))
+  (segment (start 79.8375 109.998528) (end 79.236028 110.6) (width 0.5) (layer "F.Cu") (net 6))
   (segment (start 108.633579 66.25) (end 108.057107 65.673528) (width 0.5) (layer "F.Cu") (net 6))
   (segment (start 108.05 66.8) (end 108.6 66.25) (width 0.5) (layer "F.Cu") (net 6))
@@
   (segment (start 71.6 74.275306) (end 71.6 74.7925) (width 0.25) (layer "F.Cu") (net 6))
   (segment (start 121.45 101.276472) (end 122.026472 100.7) (width 0.5) (layer "F.Cu") (net 6))
-  (segment (start 79.8375 109.998528) (end 79.236028 110.6) (width 0.5) (layer "F.Cu") (net 6))
   (segment (start 96.142489 94.175) (end 96.142489 95.2625) (width 0.3) (layer "F.Cu") (net 6))
   (segment (start 71.067055 77.872945) (end 71.07 77.87) (width 0.5) (layer "F.Cu") (net 6))
@@
   (segment (start 121.45 106.476472) (end 121.45 107.0375) (width 0.5) (layer "F.Cu") (net 6))
   (segment (start 71.962653 73.912653) (end 71.6 74.275306) (width 0.25) (layer "F.Cu") (net 6))
-  (segment (start 81.35 108.6) (end 80.488972 108.6) (width 0.5) (layer "F.Cu") (net 6))
   (segment (start 121.925 88.075) (end 122.5 88.65) (width 0.5) (layer "F.Cu") (net 6))
   (segment (start 116.475 109.0605) (end 116.475 109.948528) (width 0.5) (layer "F.Cu") (net 6))
@@
   (segment (start 121.45 101.8375) (end 121.45 101.276472) (width 0.5) (layer "F.Cu") (net 6))
   (segment (start 84.773528 68.1) (end 83.05 68.1) (width 0.5) (layer "F.Cu") (net 6))
+  (segment (start 79.236028 110.6) (end 78.675 110.6) (width 0.5) (layer "F.Cu") (net 6))
   (segment (start 96.2 108.9) (end 94.476472 108.9) (width 0.5) (layer "F.Cu") (net 6))
   (segment (start 58.1875 86.9875) (end 57.85 86.65) (width 0.5) (layer "F.Cu") (net 6))
@@
   (segment (start 85.826472 66.3) (end 85.275 66.851472) (width 0.5) (layer "F.Cu") (net 6))
   (segment (start 85.275 66.851472) (end 85.275 67.598528) (width 0.5) (layer "F.Cu") (net 6))
+  (segment (start 81.25 108.6) (end 80.488972 108.6) (width 0.5) (layer "F.Cu") (net 6))
   (segment (start 73.173528 68.1) (end 71.45 68.1) (width 0.5) (layer "F.Cu") (net 6))
   (segment (start 116.475 109.948528) (end 115.873528 110.55) (width 0.5) (layer "F.Cu") (net 6))
@@
   (segment (start 120.651053 87.574581) (end 121.151472 88.075) (width 0.5) (layer "F.Cu") (net 6))
   (segment (start 86.667489 89.722489) (end 86.675 89.73) (width 0.5) (layer "F.Cu") (net 6))
-  (segment (start 79.236028 110.6) (end 78.675 110.6) (width 0.5) (layer "F.Cu") (net 6))
   (segment (start 108.05 67.9) (end 108.05 66.8) (width 0.5) (layer "F.Cu") (net 6))
   (segment (start 108.6 66.25) (end 109.194607 66.25) (width 0.5) (layer "F.Cu") (net 6))
@@
   (segment (start 71.0875 75.805) (end 71.65 75.805) (width 0.25) (layer "F.Cu") (net 6))
   (segment (start 96.142489 82.825) (end 96.142489 80.805) (width 0.3) (layer "F.Cu") (net 6))
-  (segment (start 79.8375 109.251472) (end 79.8375 109.998528) (width 0.5) (layer "F.Cu") (net 6))
   (segment (start 117.0355 108.5) (end 116.475 109.0605) (width 0.5) (layer "F.Cu") (net 6))
   (segment (start 91.817489 89.325) (end 91.817489 89.452894) (width 0.3) (layer "F.Cu") (net 6))
   (segment (start 119.487082 106.2) (end 119.787082 105.9) (width 0.5) (layer "F.Cu") (net 6))
   (segment (start 88.325 110.75) (end 88.9 110.75) (width 0.5) (layer "F.Cu") (net 6))
-  (segment (start 80.488972 108.6) (end 79.8375 109.251472) (width 0.5) (layer "F.Cu") (net 6))
   (via (at 74.95 100.06) (size 0.8) (drill 0.4) (layers "F.Cu" "B.Cu") (free) (net 6))
   (via (at 115.25 91.3) (size 0.8) (drill 0.4) (layers "F.Cu" "B.Cu") (free) (net 6))
@@
   (via (at 127.45 89.825) (size 0.8) (drill 0.4) (layers "F.Cu" "B.Cu") (free) (net 6))
   (via (at 115.6 58.625) (size 0.8) (drill 0.4) (layers "F.Cu" "B.Cu") (net 6))
-  (via (at 88.95 108.7) (size 0.8) (drill 0.4) (layers "F.Cu" "B.Cu") (free) (net 6))
+  (via (at 88.95 108.8) (size 0.8) (drill 0.4) (layers "F.Cu" "B.Cu") (free) (net 6))
   (via (at 116.3 74.775) (size 0.8) (drill 0.4) (layers "F.Cu" "B.Cu") (free) (net 6))
   (via (at 75.15 108.8) (size 0.8) (drill 0.4) (layers "F.Cu" "B.Cu") (net 6))
@@
   (via (at 123 71.275) (size 0.8) (drill 0.4) (layers "F.Cu" "B.Cu") (free) (net 6))
   (via (at 68.15 66.2) (size 0.8) (drill 0.4) (layers "F.Cu" "B.Cu") (net 6))
-  (via (at 79.45 66.4) (size 0.8) (drill 0.4) (layers "F.Cu" "B.Cu") (net 6))
+  (via (at 79.45 67.1) (size 0.8) (drill 0.4) (layers "F.Cu" "B.Cu") (net 6))
   (via (at 124.6 76.375) (size 0.8) (drill 0.4) (layers "F.Cu" "B.Cu") (free) (net 6))
   (via (at 117.45 83.7) (size 0.8) (drill 0.4) (layers "F.Cu" "B.Cu") (free) (net 6))
@@
   (via (at 113.8 117.7) (size 0.8) (drill 0.4) (layers "F.Cu" "B.Cu") (free) (net 6))
   (via (at 108.95 60.9) (size 0.8) (drill 0.4) (layers "F.Cu" "B.Cu") (free) (net 6))
-  (via (at 90.05 108.7) (size 0.8) (drill 0.4) (layers "F.Cu" "B.Cu") (free) (net 6))
+  (via (at 90.05 108.8) (size 0.8) (drill 0.4) (layers "F.Cu" "B.Cu") (free) (net 6))
   (via (at 56.6 117.7) (size 0.8) (drill 0.4) (layers "F.Cu" "B.Cu") (free) (net 6))
-  (via (at 81.35 108.6) (size 0.8) (drill 0.4) (layers "F.Cu" "B.Cu") (free) (net 6))
+  (via (at 81.25 108.6) (size 0.8) (drill 0.4) (layers "F.Cu" "B.Cu") (free) (net 6))
   (via (at 73.95 101.01) (size 0.8) (drill 0.4) (layers "F.Cu" "B.Cu") (free) (net 6))
   (via (at 114.25 66.5) (size 0.8) (drill 0.4) (layers "F.Cu" "B.Cu") (free) (net 6))
@@
   (via (at 81.55 107.5) (size 0.8) (drill 0.4) (layers "F.Cu" "B.Cu") (net 54))
   (via (at 78.675 112.575) (size 0.8) (drill 0.4) (layers "F.Cu" "B.Cu") (net 54))
-  (segment (start 81.55 107.5) (end 81.15 107.5) (width 0.3) (layer "B.Cu") (net 54))
-  (segment (start 78.675 109.975) (end 78.675 112.575) (width 0.3) (layer "B.Cu") (net 54))
-  (segment (start 81.15 107.5) (end 78.675 109.975) (width 0.3) (layer "B.Cu") (net 54))
+  (segment (start 81.05 107.5) (end 78.675 109.875) (width 0.3) (layer "B.Cu") (net 54))
+  (segment (start 78.675 109.875) (end 78.675 112.575) (width 0.3) (layer "B.Cu") (net 54))
+  (segment (start 81.55 107.5) (end 81.05 107.5) (width 0.3) (layer "B.Cu") (net 54))
   (segment (start 86 73.51) (end 86 75.1975) (width 0.5) (layer "F.Cu") (net 55))
   (segment (start 77.45 110.1) (end 77.45 112.901472) (width 0.5) (layer "F.Cu") (net 56))
@@
         (xy 57.15 89.05)
         (xy 57.5375 89.35)
-        (xy 57.5375 90.85)
-        (xy 57.15 91.15)
-        (xy 53.9375 91.15)
-        (xy 53.6375 90.85)
+        (xy 57.5375 90.7)
+        (xy 57.15 91.05)
+        (xy 53.9375 91.05)
+        (xy 53.6375 90.7)
         (xy 53.6375 89.35)
       )

Commit message: Add files via upload
Routing:
- net INT_PI: track 54.8 -> 54.0 mm
Changed lines of the file:
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@@
   (via (at 85.15 82.2) (size 0.8) (drill 0.4) (layers "F.Cu" "B.Cu") (net 101))
   (via (at 52.65 88.45) (size 0.8) (drill 0.4) (layers "F.Cu" "B.Cu") (net 101))
-  (segment (start 51.75 84.65) (end 52.85 83.55) (width 0.3) (layer "In2.Cu") (net 101))
+  (segment (start 84.15 81.2) (end 85.15 82.2) (width 0.3) (layer "In2.Cu") (net 101))
+  (segment (start 51.75 85.9) (end 54.1 83.55) (width 0.3) (layer "In2.Cu") (net 101))
+  (segment (start 51.75 87.55) (end 51.75 85.9) (width 0.3) (layer "In2.Cu") (net 101))
+  (segment (start 62.25 81.2) (end 84.15 81.2) (width 0.3) (layer "In2.Cu") (net 101))
+  (segment (start 59.9 83.55) (end 62.25 81.2) (width 0.3) (layer "In2.Cu") (net 101))
+  (segment (start 54.1 83.55) (end 59.9 83.55) (width 0.3) (layer "In2.Cu") (net 101))
   (segment (start 52.65 88.45) (end 51.75 87.55) (width 0.3) (layer "In2.Cu") (net 101))
-  (segment (start 51.75 87.55) (end 51.75 84.65) (width 0.3) (layer "In2.Cu") (net 101))
-  (segment (start 62.25 81.2) (end 84.15 81.2) (width 0.3) (layer "In2.Cu") (net 101))
-  (segment (start 59.45 83.55) (end 59.9 83.55) (width 0.3) (layer "In2.Cu") (net 101))
-  (segment (start 84.15 81.2) (end 85.15 82.2) (width 0.3) (layer "In2.Cu") (net 101))
-  (segment (start 52.85 83.55) (end 59.45 83.55) (width 0.3) (layer "In2.Cu") (net 101))
-  (segment (start 59.9 83.55) (end 62.25 81.2) (width 0.3) (layer "In2.Cu") (net 101))
   (segment (start 106.9625 87.8) (end 106.9125 87.75) (width 0.3) (layer "F.Cu") (net 104))
   (segment (start 106.9125 87.75) (end 105.067489 87.75) (width 0.3) (layer "F.Cu") (net 104))

Commit message: Add files via upload
Parts:
- D3, D36, D4, D5: value PESD5V0U1UA -> TPESD5V0U1UA
- moved R23 2.28 mm to (88.2, 73.4)
- moved D37 2.19 mm to (88.2, 76.4)
- moved J10 1.44 mm to (125.0, 98.3)
- moved J11 1.44 mm to (125.0, 111.0)
- moved J12 1.44 mm to (125.0, 108.5)
- moved J14 1.44 mm to (125.0, 105.9)
- moved J15 1.44 mm to (125.0, 103.4)
- moved J16 1.44 mm to (125.0, 100.8)
- moved F6 1.36 mm to (120.2, 111.7), turned to 0 degrees
- moved SW1 0.92 mm to (107.5, 73.4)
- moved R11 0.90 mm to (91.3, 76.5)
- moved R7 0.90 mm to (91.3, 73.4)
- moved SW2 0.81 mm to (95.1, 73.4)
- moved U13 0.50 mm to (121.5, 106.4)
- moved TP5 0.25 mm to (61.6, 103.4)
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Connections:
- U4 pad 50: unconnected-(U4-PA15-Pad50) -> INT3
- U4 pad 54: INT3 -> unconnected-(U4-PD2-Pad54)
Routing:
- net Servo 2: track 29.8 -> 27.3 mm, vias 1 -> 0
- net INT3: track 28.4 -> 30.4 mm
- net BOOT0: track 27.6 -> 25.8 mm
- net +5VA: track 32.7 -> 31.3 mm
- net LED2: track 24.7 -> 23.4 mm
- net USB_D+: track 25.0 -> 26.2 mm
- net Servo 4: track 27.1 -> 28.3 mm
- net Servo 5: track 26.3 -> 27.3 mm
- net NRST: track 49.2 -> 48.4 mm
- net INT1: track 41.3 -> 42.1 mm
- net Servo 1: track 34.8 -> 34.2 mm
- net USB_D-: track 25.0 -> 24.5 mm
- net Servo 3: track 26.8 -> 27.3 mm
- net GND: track 66.7 -> 66.3 mm, vias 297 -> 301
- net +5V: vias 30 -> 34
Other:
- board text added: "3V3 CSN GND CE MOSI SCK MISO"
- board text added: "TESTPOINT"
- board text removed: "3V3 CSN GND CS MOSI SCK MISO"
- board text removed: "TEST"

Commit message: Add files via upload
Parts:
- moved C28 1.48 mm to (127.0, 81.2)
- moved U13 0.71 mm to (121.5, 107.1)
- moved U14 0.70 mm to (117.2, 110.5)
- moved F6 0.61 mm to (120.8, 111.8)
- moved D1 0.54 mm to (91.3, 102.3)
- moved R9 0.54 mm to (93.3, 102.3)
- moved U17 0.51 mm to (89.0, 110.8)
- moved U16 0.25 mm to (94.2, 110.7)
- moved D5 0.15 mm to (116.0, 64.7)
- moved AE1 0.09 mm to (118.2, 61.3)
- moved R10 0.06 mm to (123.0, 64.9)
Connections:
- J7 pad 6: INT5 -> GND
- J7 pad 7: GND -> INT5
- U12 pad 1: Servo 3 -> unconnected-(U12-I/O1-Pad1)
- U13 pad 1: unconnected-(U13-I/O1-Pad1) -> Servo 1
- U13 pad 3: Servo 1 -> Servo 2
- U13 pad 4: Servo 2 -> Servo 3
- U14 pad 1: MOSI -> unconnected-(U14-I/O1-Pad1)
- U15 pad 6: unconnected-(U15-I/O4-Pad6) -> MOSI
- U16 pad 1: MOSI -> unconnected-(U16-I/O1-Pad1)
- U17 pad 6: unconnected-(U17-I/O4-Pad6) -> MOSI
- U4 pad 33: Servo 2 -> unconnected-(U4-PB12-Pad33)
- U4 pad 34: Servo 3 -> Servo 2
- U4 pad 35: Servo 4 -> Servo 3
- U4 pad 36: Servo 5 -> Servo 4
- U4 pad 37: ESC -> Servo 5
- U4 pad 38: INT_GPS -> ESC
- U4 pad 39: FLASH_CS -> INT_GPS
- U4 pad 40: CS_EXTRA -> FLASH_CS
- U4 pad 41: unconnected-(U4-PA8-Pad41) -> CS_EXTRA
Routing:
- net CSN: track 31.2 -> 39.0 mm, vias 2 -> 0
- net INT4: track 33.4 -> 39.3 mm
- net GND: track 66.3 -> 71.8 mm, vias 301 -> 323
- net CS_EXTRA: track 32.2 -> 37.6 mm, vias 4 -> 2
- net INT5: track 34.9 -> 38.9 mm
- net INT_GPS: track 58.5 -> 62.1 mm
- net Servo 2: track 27.3 -> 30.8 mm, vias 0 -> 1
- net SCK: track 57.6 -> 54.4 mm, vias 3 -> 2
- net MOSI: track 61.1 -> 63.8 mm, vias 4 -> 2
- net Servo 4: track 28.3 -> 26.2 mm, vias 1 -> 0
- net Servo 1: track 34.2 -> 32.2 mm
- net Net-(U6-VCC_RF): track 8.21 -> 9.43 mm, vias 0 -> 2
- net INT1: track 42.1 -> 43.2 mm
- net Servo 3: track 27.3 -> 26.4 mm
- net MISO: track 55.9 -> 56.8 mm
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Other:
- board text added: "3V3 CS SCK MOSI MISO GND INT"
- board text removed: "3V3 CS SCK MOSI MISO INT GND"
