File: FlightComputer.kicad_pcb (KiCad board)
At the start: 4 copper layers, 83 x 62 mm, 131 parts, among them IC1 LMR33640DDDAR, J1 SM05B-GHS-TB, J10 Header1x3Pin, J11 Header1x3Pin, J12 Header1x3Pin, J13 SM02B-GHS-TB, J14 Header1x3Pin, J15 Header1x3Pin, J16 Header1x3Pin, J17 SM02B-GHS-TB, J18 USB_C_Receptacle, J19 SM02B-GHS-TB, J2 Screw_Terminal_01x02, J3 SM07B-GHS-TB, J4 SM05B-GHS-TB, J5 SM07B-GHS-TB, J6 SM05B-GHS-TB, J7 SM07B-GHS-TB, J8 SM05B-GHS-TB, J9 SM05B-GHS-TB, Q1 SI2369BDS-T1-GE3 30V 5.6A, SW1 KMR221GLFS, SW2 KMR221GLFS, U1 LIS3MDL, U10 USBLC6-4SC6, U11 USBLC6-4SC6, U12 USBLC6-4SC6, U13 USBLC6-4SC6, U14 USBLC6-4SC6, U15 USBLC6-4SC6, U16 USBLC6-4SC6, U17 USBLC6-4SC6, U18 USBLC6-4SC6, U19 USBLC6-4SC6, U2 BMI270, U20 USBLC6-4SC6, U3 AP7361C-33ER-13, U4 STM32F446RET6, U5 LPS22HH, U6 NEO-M9N, U7 W25Q128JVSIQ, U8 USBLC6-4SC6, U9 USBLC6-4SC6, Y1 16MHz

Commit message: Add files via upload
Parts:
- moved R9 0.22 mm to (93.2, 102.5)
- moved D1 0.20 mm to (91.3, 102.5)
Routing:
- net V_BAT_SENSE: track 68.0 -> 68.7 mm
- net INT4: track 39.3 -> 39.9 mm
- net GND: vias 323 -> 327

Commit message: Add files via upload
Routing:
- net GND: vias 327 -> 328
Changed lines of the file:
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@@
   (via (at 130.35 74.4) (size 0.8) (drill 0.4) (layers "F.Cu" "B.Cu") (free) (net 6))
   (via (at 104.55 70.4) (size 0.8) (drill 0.4) (layers "F.Cu" "B.Cu") (net 6))
-  (via (at 101.05 76.2) (size 0.8) (drill 0.4) (layers "F.Cu" "B.Cu") (free) (net 6))
+  (via (at 101.15 76.3) (size 0.8) (drill 0.4) (layers "F.Cu" "B.Cu") (free) (net 6))
   (via (at 82.25 96.2) (size 0.8) (drill 0.4) (layers "F.Cu" "B.Cu") (free) (net 6))
   (via (at 124.65 76.3) (size 0.8) (drill 0.4) (layers "F.Cu" "B.Cu") (free) (net 6))
@@
   (via (at 115.75 72.5) (size 0.8) (drill 0.4) (layers "F.Cu" "B.Cu") (free) (net 6))
   (via (at 55.275 77) (size 0.8) (drill 0.4) (layers "F.Cu" "B.Cu") (net 6))
+  (via (at 123.45 101.8) (size 0.8) (drill 0.4) (layers "F.Cu" "B.Cu") (free) (net 6))
   (via (at 69.95 63.4) (size 0.8) (drill 0.4) (layers "F.Cu" "B.Cu") (free) (net 6))
   (via (at 60.613 97.7) (size 0.8) (drill 0.4) (layers "F.Cu" "B.Cu") (free) (net 6))
@@
   (via (at 120.85 62.1) (size 0.8) (drill 0.4) (layers "F.Cu" "B.Cu") (free) (net 6))
   (via (at 77.3475 73.945) (size 0.8) (drill 0.4) (layers "F.Cu" "B.Cu") (free) (net 6))
-  (via (at 102.25 76.2) (size 0.8) (drill 0.4) (layers "F.Cu" "B.Cu") (free) (net 6))
+  (via (at 102.15 76.3) (size 0.8) (drill 0.4) (layers "F.Cu" "B.Cu") (free) (net 6))
   (via (at 117.15 90.3) (size 0.8) (drill 0.4) (layers "F.Cu" "B.Cu") (free) (net 6))
   (via (at 118.8 58.6) (size 0.8) (drill 0.4) (layers "F.Cu" "B.Cu") (net 6))
@@
   (segment (start 108.75 104.7) (end 107.25 103.2) (width 0.3) (layer "F.Cu") (net 10))
   (segment (start 101.135 114.965) (end 99.84 114.965) (width 0.3) (layer "F.Cu") (net 10))
+  (segment (start 114.035 110.186472) (end 114.035 113.9) (width 0.5) (layer "F.Cu") (net 11))
   (segment (start 108.45 116.236472) (end 109.286472 115.4) (width 0.3) (layer "F.Cu") (net 11))
   (segment (start 109.286472 115.4) (end 110.35 115.4) (width 0.3) (layer "F.Cu") (net 11))
-  (segment (start 112.8875 109.6) (end 113.448528 109.6) (width 0.5) (layer "F.Cu") (net 11))
+  (segment (start 112.8875 109.6) (end 113.65 109.6) (width 0.5) (layer "F.Cu") (net 11))
   (segment (start 112.85 116.2) (end 114.035 115.015) (width 0.3) (layer "F.Cu") (net 11))
   (segment (start 91.2375 110.3) (end 91.2375 108.2125) (width 0.3) (layer "F.Cu") (net 11))
-  (segment (start 100.775 100.125) (end 102.85 102.2) (width 0.3) (layer "F.Cu") (net 11))
-  (segment (start 109.35 102.2) (end 114.05 106.9) (width 0.3) (layer "F.Cu") (net 11))
-  (segment (start 114.05 106.9) (end 114.05 108.998528) (width 0.3) (layer "F.Cu") (net 11))
+  (segment (start 114.035 109.985) (end 114.035 106.885) (width 0.3) (layer "F.Cu") (net 11))
+  (segment (start 113.65 109.6) (end 114.035 109.985) (width 0.5) (layer "F.Cu") (net 11))
   (segment (start 107.945 117.505) (end 108.45 117) (width 0.3) (layer "F.Cu") (net 11))
   (segment (start 91.2375 110.3) (end 90.7375 109.8) (width 0.5) (layer "F.Cu") (net 11))
@@
   (segment (start 91.2375 111.5875) (end 91.75 112.1) (width 0.5) (layer "F.Cu") (net 11))
   (segment (start 90.7375 109.8) (end 90.0875 109.8) (width 0.5) (layer "F.Cu") (net 11))
+  (segment (start 102.85 102.2) (end 100.775 100.125) (width 0.3) (layer "F.Cu") (net 11))
   (segment (start 91.2375 108.2125) (end 96.65 102.8) (width 0.3) (layer "F.Cu") (net 11))
   (segment (start 111.15 116.2) (end 112.85 116.2) (width 0.3) (layer "F.Cu") (net 11))
   (segment (start 100.775 100.125) (end 98.642489 97.992489) (width 0.3) (layer "F.Cu") (net 11))
-  (segment (start 114.05 108.998528) (end 113.448528 109.6) (width 0.3) (layer "F.Cu") (net 11))
+  (segment (start 114.035 109.985) (end 114.035 110.186472) (width 0.5) (layer "F.Cu") (net 11))
+  (segment (start 114.035 106.885) (end 109.35 102.2) (width 0.3) (layer "F.Cu") (net 11))
   (segment (start 107.04 117.505) (end 107.945 117.505) (width 0.3) (layer "F.Cu") (net 11))
   (segment (start 110.35 115.4) (end 111.15 116.2) (width 0.3) (layer "F.Cu") (net 11))
   (segment (start 96.65 102.8) (end 96.65 99.4) (width 0.3) (layer "F.Cu") (net 11))
-  (segment (start 114.035 110.186472) (end 114.035 113.9) (width 0.5) (layer "F.Cu") (net 11))
   (segment (start 98.642489 97.992489) (end 98.642489 94.175) (width 0.3) (layer "F.Cu") (net 11))
-  (segment (start 113.448528 109.6) (end 114.035 110.186472) (width 0.5) (layer "F.Cu") (net 11))
   (segment (start 91.2375 110.3) (end 91.2375 111.5875) (width 0.5) (layer "F.Cu") (net 11))
-  (segment (start 102.85 102.2) (end 109.35 102.2) (width 0.3) (layer "F.Cu") (net 11))
   (segment (start 108.45 117) (end 108.45 116.236472) (width 0.3) (layer "F.Cu") (net 11))
+  (segment (start 109.35 102.2) (end 102.85 102.2) (width 0.3) (layer "F.Cu") (net 11))
   (segment (start 114.035 115.015) (end 114.035 113.9) (width 0.3) (layer "F.Cu") (net 11))
   (via (at 100.775 100.125) (size 0.8) (drill 0.4) (layers "F.Cu" "B.Cu") (net 11))
@@
   (via (at 99.65 102.4) (size 0.8) (drill 0.4) (layers "F.Cu" "B.Cu") (net 74))
   (via (at 101.257719 92.1) (size 0.8) (drill 0.4) (layers "F.Cu" "B.Cu") (net 74))
-  (segment (start 101.257719 92.392281) (end 101.257719 92.1) (width 0.3) (layer "B.Cu") (net 74))
-  (segment (start 99.65 94) (end 101.257719 92.392281) (width 0.3) (layer "B.Cu") (net 74))
-  (segment (start 99.65 102.4) (end 99.65 94) (width 0.3) (layer "B.Cu") (net 74))
+  (segment (start 99.65 102.4) (end 99.65 94.2) (width 0.3) (layer "B.Cu") (net 74))
+  (segment (start 101.257719 92.592281) (end 101.257719 92.1) (width 0.3) (layer "B.Cu") (net 74))
+  (segment (start 99.65 94.2) (end 101.257719 92.592281) (width 0.3) (layer "B.Cu") (net 74))
   (segment (start 122.975 91.4) (end 124.605 89.77) (width 0.3) (layer "F.Cu") (net 77))
   (segment (start 124.605 89.77) (end 125.323949 89.77) (width 0.3) (layer "F.Cu") (net 77))
@@
   (segment (start 96.95 72.8) (end 97.15 72.6) (width 0.5) (layer "F.Cu") (net 83))
   (segment (start 92.245 72.58) (end 93.03 72.58) (width 0.5) (layer "F.Cu") (net 83))
+  (segment (start 97.642489 84) (end 97.642489 82.825) (width 0.3) (layer "F.Cu") (net 83))
   (segment (start 91.35 72.575) (end 91.355 72.58) (width 0.5) (layer "F.Cu") (net 83))
+  (segment (start 89.75 81) (end 90.7 81.95) (width 0.3) (layer "F.Cu") (net 83))
+  (segment (start 97.242489 84.4) (end 97.642489 84) (width 0.3) (layer "F.Cu") (net 83))
   (segment (start 95.392489 84.4) (end 97.242489 84.4) (width 0.3) (layer "F.Cu") (net 83))
+  (segment (start 91.355 72.58) (end 92.245 72.58) (width 0.5) (layer "F.Cu") (net 83))
+  (segment (start 93.05 72.6) (end 93.25 72.8) (width 0.5) (layer "F.Cu") (net 83))
+  (segment (start 89.75 73.4) (end 89.75 81) (width 0.3) (layer "F.Cu") (net 83))
+  (segment (start 91.35 72.575) (end 90.575 72.575) (width 0.3) (layer "F.Cu") (net 83))
+  (segment (start 90.575 72.575) (end 89.75 73.4) (width 0.3) (layer "F.Cu") (net 83))
   (segment (start 90.7 81.95) (end 92.942489 81.95) (width 0.3) (layer "F.Cu") (net 83))
+  (segment (start 93.25 72.8) (end 96.95 72.8) (width 0.5) (layer "F.Cu") (net 83))
   (segment (start 92.942489 81.95) (end 95.392489 84.4) (width 0.3) (layer "F.Cu") (net 83))
-  (segment (start 91.355 72.58) (end 92.245 72.58) (width 0.5) (layer "F.Cu") (net 83))
-  (segment (start 97.642489 84) (end 97.642489 82.825) (width 0.3) (layer "F.Cu") (net 83))
-  (segment (start 93.05 72.6) (end 93.25 72.8) (width 0.5) (layer "F.Cu") (net 83))
-  (segment (start 91.35 72.575) (end 89.65 74.275) (width 0.3) (layer "F.Cu") (net 83))
-  (segment (start 93.25 72.8) (end 96.95 72.8) (width 0.5) (layer "F.Cu") (net 83))
-  (segment (start 97.242489 84.4) (end 97.642489 84) (width 0.3) (layer "F.Cu") (net 83))
-  (segment (start 89.65 80.9) (end 90.7 81.95) (width 0.3) (layer "F.Cu") (net 83))
-  (segment (start 89.65 74.275) (end 89.65 80.9) (width 0.3) (layer "F.Cu") (net 83))
   (segment (start 93.03 72.58) (end 93.05 72.6) (width 0.3) (layer "F.Cu") (net 83))
   (segment (start 91.35 75.625) (end 91.35 74.225) (width 0.5) (layer "F.Cu") (net 87))
@@
   (segment (start 82.7 64.25) (end 82.7 62.75) (width 0.5) (layer "F.Cu") (net 94))
   (segment (start 82.35 65.5) (end 83.15 66.3) (width 0.5) (layer "F.Cu") (net 94))
-  (segment (start 118.2875 110.55) (end 118.848528 110.55) (width 0.5) (layer "F.Cu") (net 95))
+  (segment (start 119.9625 111.4125) (end 119.9625 112.9725) (width 0.5) (layer "F.Cu") (net 95))
+  (segment (start 119.1 110.55) (end 119.9625 111.4125) (width 0.5) (layer "F.Cu") (net 95))
+  (segment (start 118.2875 110.55) (end 119.1 110.55) (width 0.5) (layer "F.Cu") (net 95))
   (segment (start 119.9625 112.9725) (end 119.035 113.9) (width 0.5) (layer "F.Cu") (net 95))
-  (segment (start 118.848528 110.55) (end 119.9625 111.663972) (width 0.5) (layer "F.Cu") (net 95))
-  (segment (start 119.9625 111.663972) (end 119.9625 112.9725) (width 0.5) (layer "F.Cu") (net 95))
   (segment (start 97.15 112.25) (end 95.5 113.9) (width 0.5) (layer "F.Cu") (net 96))
   (segment (start 96.35 110.7) (end 97.15 111.5) (width 0.5) (layer "F.Cu") (net 96))
@@
   (via (at 88.15 78.2125) (size 0.8) (drill 0.4) (layers "F.Cu" "B.Cu") (net 108))
   (via (at 101.25 87.25) (size 0.8) (drill 0.4) (layers "F.Cu" "B.Cu") (net 108))
-  (segment (start 101.1 87.1) (end 101.25 87.25) (width 0.3) (layer "B.Cu") (net 108))
-  (segment (start 94.134339 87.1) (end 101.1 87.1) (width 0.3) (layer "B.Cu") (net 108))
+  (segment (start 88.15 81.115661) (end 94.284339 87.25) (width 0.3) (layer "B.Cu") (net 108))
   (segment (start 88.15 78.2125) (end 88.15 81.115661) (width 0.3) (layer "B.Cu") (net 108))
-  (segment (start 88.15 81.115661) (end 94.134339 87.1) (width 0.3) (layer "B.Cu") (net 108))
+  (segment (start 94.284339 87.25) (end 101.25 87.25) (width 0.3) (layer "B.Cu") (net 108))
   (segment (start 73.2 109.9) (end 71.85 109.9) (width 0.5) (layer "F.Cu") (net 110))
   (segment (start 81.75 113.9) (end 81.75 112.5375) (width 0.5) (layer "F.Cu") (net 111))

Commit message: Add files via upload
Parts:
- moved C28 1.12 mm to (128.1, 81.7), turned to -90 degrees
- moved R19 0.30 mm to (94.2, 78.9)
- moved R20 0.30 mm to (103.5, 78.9)
- moved R6 0.30 mm to (97.3, 78.9)
- moved R8 0.30 mm to (100.5, 78.9)
- moved R11 0.28 mm to (91.5, 76.7)
- moved R7 0.28 mm to (91.5, 73.6)
- moved D37 0.26 mm to (88.0, 76.7)
- moved R23 0.20 mm to (88.0, 73.6)
- moved SW1 0.20 mm to (107.5, 73.6)
- moved SW2 0.20 mm to (95.1, 73.6)
- moved C2 0.10 mm to (92.3, 80.9)
- moved C7 0.10 mm to (95.4, 80.9)
- moved AE1 0.10 mm to (118.2, 61.2)
Routing:
- net GND: track 71.8 -> 64.5 mm, vias 328 -> 326
- net INT1: track 43.2 -> 40.7 mm
- net SDA: track 115.0 -> 113.6 mm
- net SCL: track 99.6 -> 98.5 mm
- net INT2: track 33.9 -> 34.6 mm
- net INT3: track 30.4 -> 29.8 mm
- net USART3_TX: track 29.2 -> 29.7 mm
Other:
- board text added: "change d37 to d10 or someting"

Commit message: Add files via upload
Parts:
- moved C25 0.70 mm to (106.8, 83.6)
- moved SW1 0.63 mm to (106.8, 73.8)
- moved C32 0.50 mm to (102.2, 75.0)
- moved SW2 0.40 mm to (95.5, 73.8)
- moved C4 0.40 mm to (72.2, 77.8)
- moved C5 0.40 mm to (63.3, 75.4)
- moved C6 0.40 mm to (65.7, 78.1)
- moved U1 0.40 mm to (72.2, 75.5)
- moved U5 0.40 mm to (78.9, 75.5)
- moved C1 0.40 mm to (74.5, 77.0)
- moved C17 0.40 mm to (81.1, 75.5)
- moved C3 0.40 mm to (74.5, 74.1)
- moved U2 0.40 mm to (65.6, 75.5)
- moved C2 0.35 mm to (92.6, 80.9)
- moved C21 0.30 mm to (103.2, 96.2)
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- renumbered D37 to D6, D35 to D7, D36 to D8
Routing:
- net GND: track 64.5 -> 72.5 mm, vias 326 -> 323
- net NRST: track 48.5 -> 53.6 mm
- net SCL: track 98.5 -> 97.5 mm
- net +5V: vias 34 -> 36
Other:
- board text removed: "PAYLOAD"
- board text removed: "change d37 to d10 or someting"

Commit message: Add files via upload
Connections:
- U4 pad 39: INT_GPS -> unconnected-(U4-PC8-Pad39)
- U6 pad 4: INT_GPS -> unconnected-(U6-EXTINT-Pad4)
Routing:
- net INT_GPS: track 62.1 -> 0.00 mm
- net GND: vias 323 -> 330
Other:
- board text added: "use 28 and 25 for flash cs"

Commit message: Add files via upload
Parts:
- added D9: GREEN, LED_SMD:LED_0603_1608Metric, F.Cu at (118.7, 95.3)
- added R25: 1k, Resistor_SMD:R_0603_1608Metric, F.Cu at (121.8, 95.3)
- D1: value GREEN -> RED
- D2, D6: value RED -> GREEN
- moved C1 0.20 mm to (74.5, 76.8)
- moved C17 0.20 mm to (81.1, 75.3)
- moved C5 0.20 mm to (63.3, 75.2)
- moved C6 0.20 mm to (65.7, 77.9)
- moved SW1 0.20 mm to (106.8, 74.0)
- moved SW2 0.20 mm to (95.5, 74.0)
- moved U2 0.20 mm to (65.6, 75.3)
- moved U5 0.20 mm to (78.9, 75.3)
- moved C3 0.20 mm to (74.5, 73.9)
- moved C4 0.20 mm to (72.2, 77.6)
- moved U1 0.20 mm to (72.2, 75.3)
- moved C19 0.16 mm to (91.8, 83.8)
- moved C30 0.10 mm to (91.8, 90.1)
Connections:
- U4 pad 39: unconnected-(U4-PC8-Pad39) -> LED3
Routing:
- net LED3: track 0.00 -> 15.3 mm
- net Net-(D9-K): track 0.00 -> 1.58 mm
- net GND: track 72.5 -> 73.5 mm, vias 330 -> 325
Other:
- board text added: "STATUS3"
- board text removed: "use 28 and 25 for flash cs"

Commit message: Add files via upload
Parts:
- moved C19 0.45 mm to (91.3, 83.8)
- moved C2 0.45 mm to (92.2, 80.9)
- moved C20 0.45 mm to (87.0, 89.7)
- moved C21 0.45 mm to (102.8, 96.2)
- moved C22 0.45 mm to (105.2, 94.6)
- moved C24 0.45 mm to (95.4, 96.2)
- moved C25 0.45 mm to (106.3, 83.6)
- moved C30 0.45 mm to (91.3, 90.1)
- moved C32 0.45 mm to (101.8, 75.0)
- moved C7 0.45 mm to (95.2, 80.9)
- moved D2 0.45 mm to (107.3, 87.8)
- moved D6 0.45 mm to (87.8, 76.8)
- moved L2 0.45 mm to (87.0, 91.4)
- moved R1 0.45 mm to (90.5, 87.7)
- moved R11 0.45 mm to (91.3, 76.8)
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Routing:
- net UART4_TX: track 51.8 -> 50.3 mm
- net NRST: track 53.3 -> 54.7 mm
- net SWO: track 24.4 -> 25.3 mm
- net INT1: track 40.7 -> 39.9 mm
- net +5V: track 27.4 -> 28.2 mm
- net GND: vias 325 -> 326
Other:
- board text added: "5V PWR"
