File: FlightComputer.kicad_pcb (KiCad board)
At the start: 4 copper layers, 83 x 62 mm, 133 parts, among them IC1 LMR33640DDDAR, J1 SM05B-GHS-TB, J10 Header1x3Pin, J11 Header1x3Pin, J12 Header1x3Pin, J13 SM02B-GHS-TB, J14 Header1x3Pin, J15 Header1x3Pin, J16 Header1x3Pin, J17 SM02B-GHS-TB, J18 USB_C_Receptacle, J19 SM02B-GHS-TB, J2 Screw_Terminal_01x02, J3 SM07B-GHS-TB, J4 SM05B-GHS-TB, J5 SM07B-GHS-TB, J6 SM05B-GHS-TB, J7 SM07B-GHS-TB, J8 SM05B-GHS-TB, J9 SM05B-GHS-TB, Q1 SI2369BDS-T1-GE3 30V 5.6A, SW1 KMR221GLFS, SW2 KMR221GLFS, U1 LIS3MDL, U10 USBLC6-4SC6, U11 USBLC6-4SC6, U12 USBLC6-4SC6, U13 USBLC6-4SC6, U14 USBLC6-4SC6, U15 USBLC6-4SC6, U16 USBLC6-4SC6, U17 USBLC6-4SC6, U18 USBLC6-4SC6, U19 USBLC6-4SC6, U2 BMI270, U20 USBLC6-4SC6, U3 AP7361C-33ER-13, U4 STM32F446RET6, U5 LPS22HH, U6 NEO-M9N, U7 W25Q128JVSIQ, U8 USBLC6-4SC6, U9 USBLC6-4SC6, Y1 16MHz

Commit message: Add files via upload
Parts:
- added TP6: TestPoint, TestPoint:TestPoint_Pad_D1.5mm, F.Cu at (113.5, 79.7)
- moved C32 1.07 mm to (100.7, 75.0)
- moved C29 0.89 mm to (88.8, 90.1)
- moved C9 0.89 mm to (86.1, 83.7)
- moved SW1 0.89 mm to (105.5, 74.0)
- moved C19 0.89 mm to (90.4, 83.8)
- moved C2 0.89 mm to (91.3, 80.9)
- moved C20 0.89 mm to (86.1, 89.7)
- moved C21 0.89 mm to (101.9, 96.2)
- moved C22 0.89 mm to (104.3, 94.6)
- moved C24 0.89 mm to (94.5, 96.2)
- moved C25 0.89 mm to (105.4, 83.6)
- moved C30 0.89 mm to (90.4, 90.1)
- moved C7 0.89 mm to (94.3, 80.9)
- moved D2 0.89 mm to (106.4, 87.8)
- moved D6 0.89 mm to (86.9, 76.8)
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Connections:
- U6 pad 1: unconnected-(U6-SAFEBOOT_N-Pad1) -> Net-(U6-SAFEBOOT_N)
Routing:
- net Net-(U6-SAFEBOOT_N): track 0.00 -> 32.1 mm, vias 0 -> 2
- net SDA: track 113.0 -> 114.6 mm
- net USART3_TX: track 29.3 -> 30.6 mm
- net USART3_RX: track 29.1 -> 30.5 mm
- net MISO: track 57.2 -> 58.4 mm
- net INT4: track 39.4 -> 38.4 mm
- net INT5: track 39.1 -> 38.2 mm
- net INT1: track 39.9 -> 39.1 mm
- net USB_D-: track 24.9 -> 25.8 mm
- net USB_D+: track 26.7 -> 27.6 mm
- net Servo 5: track 28.0 -> 28.9 mm
- net Servo 3: track 26.8 -> 27.7 mm
- net Servo 2: track 31.2 -> 32.1 mm
- net LED3: track 15.8 -> 16.7 mm
- net ESC: track 25.1 -> 26.0 mm
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Other:
- board text added: "SAFE"
- board text removed: "5V PWR"

Commit message: Add files via upload
Parts:
- TP6: footprint TestPoint:TestPoint_Pad_D1.5mm -> TestPoint:TestPoint_Keystone_5000-5004_Miniature
- moved C28 2.21 mm to (130.2, 81.0), turned to 0 degrees
- moved TP6 0.65 mm to (112.8, 79.4)
- moved R12 0.26 mm to (109.8, 87.8)
Connections:
- U1 pad 8: unconnected-(U1-DRDY-Pad8) -> INT_MAG
- U4 pad 33: unconnected-(U4-PB12-Pad33) -> INT_MAG
Routing:
- net INT_MAG: track 0.00 -> 52.5 mm, vias 0 -> 2
- net INT_BARO: track 25.4 -> 34.3 mm
- net Net-(U6-SAFEBOOT_N): track 32.1 -> 30.9 mm, vias 2 -> 1
- net GND: track 73.5 -> 74.5 mm, vias 322 -> 332
- net USART3_TX: track 30.6 -> 31.2 mm
- net USART3_RX: track 30.5 -> 31.0 mm
Other:
- board text added: "get rid of the 5v pour https://www.ti.com/lit/ug/snvu664/snvu664.pdf?ts=1689743743891&ref_url=https%253A%252F%252Fwww.google.com%252F"

Commit message: Add files via upload
Parts:
- moved TP1 0.40 mm to (70.3, 83.4)
- moved TP4 0.40 mm to (77.8, 83.4)
- moved TP3 0.40 mm to (62.8, 83.4)
Routing:
- net GND: vias 332 -> 335
Other:
- board text added: "5V1"
- board text removed: "5V"
- board text removed: "get rid of the 5v pour https://www.ti.com/lit/ug/snvu664/snvu664.pdf?ts=1689743743891&ref_url=https%253A%252F%252Fwww.google.com%252F"
Changed lines of the file:
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@@
   )
   (footprint "TestPoint:TestPoint_Keystone_5000-5004_Miniature" (layer "F.Cu")
-    (at 78.25 83.4 180)
+    (at 77.85 83.4 180)
     (descr "Keystone Miniature THM Test Point 5000-5004, http://www.keyelco.com/product-pdf.cfm?p=1309")
     (tags "Through Hole Mount Test Points")
@@
   )
   (footprint "TestPoint:TestPoint_Keystone_5000-5004_Miniature" (layer "F.Cu")
-    (at 70.7 83.4)
+    (at 70.3 83.4)
     (descr "Keystone Miniature THM Test Point 5000-5004, http://www.keyelco.com/product-pdf.cfm?p=1309")
     (tags "Through Hole Mount Test Points")
@@
   )
   (footprint "TestPoint:TestPoint_Keystone_5000-5004_Miniature" (layer "F.Cu")
-    (at 63.15 83.4)
+    (at 62.75 83.4)
     (descr "Keystone Miniature THM Test Point 5000-5004, http://www.keyelco.com/product-pdf.cfm?p=1309")
     (tags "Through Hole Mount Test Points")
@@
   (gr_line (start 128.85 116.6) (end 128.9 88.7)
     (stroke (width 0.1) (type default)) (layer "F.Fab"))
-  (gr_text "get rid of the 5v pour\nhttps://www.ti.com/lit/ug/snvu664/snvu664.pdf?ts=1689743743891&ref_url=https%253A%252F%252Fwww.google.com%252F" (at 23.55 125.9) (layer "F.Cu")
-    (effects (font (size 1.5 1.5) (thickness 0.3) bold) (justify left bottom))
-  )
   (gr_text "GND\nINT\nSDA\nSCL\n3V3" (at 69.95 59.18 270) (layer "B.SilkS")
     (effects (font (size 1 1) (thickness 0.15)) (justify right bottom mirror))
@@
     (effects (font (size 1 1) (thickness 0.15)))
   )
-  (gr_text "3V3" (at 80.6 84.15) (layer "F.SilkS")
+  (gr_text "3V3" (at 80.2 84.05) (layer "F.SilkS")
     (effects (font (size 1 1) (thickness 0.15)) (justify left bottom))
   )
@@
     (effects (font (size 1 1) (thickness 0.15)) (justify left bottom))
   )
-  (gr_text "GND" (at 72.95 84.05) (layer "F.SilkS")
+  (gr_text "GND" (at 72.55 84.05) (layer "F.SilkS")
     (effects (font (size 1 1) (thickness 0.15)) (justify left bottom))
   )
@@
     (effects (font (size 1 1) (thickness 0.15)))
   )
-  (gr_text "5V" (at 65.45 84) (layer "F.SilkS")
+  (gr_text "5V1" (at 65.05 84) (layer "F.SilkS")
     (effects (font (size 1 1) (thickness 0.15)) (justify left bottom))
   )
@@
   (segment (start 82.65 114.7) (end 67.1 114.7) (width 0.5) (layer "B.Cu") (net 1))
   (segment (start 67.1 114.7) (end 54.5 102.1) (width 0.5) (layer "B.Cu") (net 1))
-  (segment (start 63.15 83.4) (end 57.9 83.4) (width 1) (layer "F.Cu") (net 3))
   (segment (start 77.1 107.91) (end 77.1 106.977) (width 0.5) (layer "F.Cu") (net 3))
+  (segment (start 62.75 83.4) (end 57.9 83.4) (width 1) (layer "F.Cu") (net 3))
   (via (at 59.45 91.7) (size 0.8) (drill 0.4) (layers "F.Cu" "B.Cu") (net 3))
   (via (at 55.55 67.5) (size 0.8) (drill 0.4) (layers "F.Cu" "B.Cu") (free) (net 3))
@@
   (via (at 116.6 63.1) (size 0.8) (drill 0.4) (layers "F.Cu" "B.Cu") (free) (net 6))
   (via (at 105.365 110.4) (size 0.8) (drill 0.4) (layers "F.Cu" "B.Cu") (free) (net 6))
+  (via (at 74.45 103.1) (size 0.8) (drill 0.4) (layers "F.Cu" "B.Cu") (free) (net 6))
   (via (at 74.95 97.1) (size 0.8) (drill 0.4) (layers "F.Cu" "B.Cu") (free) (net 6))
   (via (at 110.95 84.4) (size 0.8) (drill 0.4) (layers "F.Cu" "B.Cu") (free) (net 6))
@@
   (via (at 115.6 58.625) (size 0.8) (drill 0.4) (layers "F.Cu" "B.Cu") (net 6))
   (via (at 88.4375 108.8) (size 0.8) (drill 0.4) (layers "F.Cu" "B.Cu") (free) (net 6))
+  (via (at 83.65 96) (size 0.8) (drill 0.4) (layers "F.Cu" "B.Cu") (free) (net 6))
   (via (at 74.75 108.8) (size 0.8) (drill 0.4) (layers "F.Cu" "B.Cu") (net 6))
   (via (at 64.45 113.6) (size 0.8) (drill 0.4) (layers "F.Cu" "B.Cu") (net 6))
@@
   (via (at 118.95 72.5) (size 0.8) (drill 0.4) (layers "F.Cu" "B.Cu") (free) (net 6))
   (via (at 75.35 111.6) (size 0.8) (drill 0.4) (layers "F.Cu" "B.Cu") (net 6))
+  (via (at 79.15 65.5) (size 0.8) (drill 0.4) (layers "F.Cu" "B.Cu") (free) (net 6))
   (via (at 60.871899 62.5) (size 0.8) (drill 0.4) (layers "F.Cu" "B.Cu") (free) (net 6))
   (via (at 128.85 88.218121) (size 0.8) (drill 0.4) (layers "F.Cu" "B.Cu") (free) (net 6))
@@
   (segment (start 83.95 64.3) (end 83.95 65.1875) (width 0.5) (layer "F.Cu") (net 7))
   (segment (start 72.5125 64.3) (end 72.5125 62.8125) (width 0.5) (layer "F.Cu") (net 7))
-  (segment (start 69.35 69.5) (end 67.95375 70.89625) (width 0.25) (layer "F.Cu") (net 7))
   (segment (start 69.9875 76.075) (end 70.7 76.075) (width 0.25) (layer "F.Cu") (net 7))
-  (segment (start 67.95375 70.89625) (end 67.95375 74.0805) (width 0.25) (layer "F.Cu") (net 7))
   (segment (start 98.161883 80.888117) (end 97.3 81.75) (width 0.3) (layer "F.Cu") (net 7))
   (segment (start 98.707511 77.196245) (end 98.161883 77.741873) (width 0.25) (layer "F.Cu") (net 7))
@@
   (segment (start 77.835 71.8) (end 77.835 74.5375) (width 0.25) (layer "F.Cu") (net 7))
   (segment (start 77.85 69.5) (end 97.307511 69.5) (width 0.25) (layer "F.Cu") (net 7))
+  (segment (start 67.95375 70.89625) (end 67.95375 74.0805) (width 0.25) (layer "F.Cu") (net 7))
+  (segment (start 69.35 69.5) (end 67.95375 70.89625) (width 0.25) (layer "F.Cu") (net 7))
   (segment (start 95.3625 62.7875) (end 95.4 62.75) (width 0.3) (layer "F.Cu") (net 7))
   (segment (start 83.95 65.1875) (end 84.1125 65.35) (width 0.3) (layer "F.Cu") (net 7))
   (segment (start 98.161883 78.9) (end 98.161883 80.888117) (width 0.3) (layer "F.Cu") (net 7))
   (segment (start 95.3625 65.25) (end 95.4625 65.35) (width 0.5) (layer "F.Cu") (net 7))
-  (segment (start 77.85 69.5) (end 69.35 69.5) (width 0.25) (layer "F.Cu") (net 7))
   (segment (start 95.3625 64.3375) (end 95.3625 65.25) (width 0.5) (layer "F.Cu") (net 7))
+  (segment (start 77.85 69.5) (end 69.35 69.5) (width 0.25) (layer "F.Cu") (net 7))
   (segment (start 95.3625 64.3375) (end 95.3625 62.7875) (width 0.5) (layer "F.Cu") (net 7))
   (segment (start 65.76 75.3) (end 69.2125 75.3) (width 0.25) (layer "F.Cu") (net 7))
