File: Microcontroller.kicad_sch (KiCad schematic)
At the start: 31 parts, among them SW1 KMR221GLFS, U4 STM32F446RET6, U7 W25Q128JVSIQ, Y1 16MHz

Commit message: Add files via upload
Connections:
- net INT5: now reaches U4.10 (PC2)
- net INT4: now reaches U4.11 (PC3)
- net INT1: now reaches U4.2 (PC13)
- net INT2: now reaches U4.4 (PC15)
- net INT3: now reaches U4.54 (PD2)
- no-connect marks 17 -> 12
Other:
- moved on the sheet: D1, R9

Commit message: Add files via upload
Changed lines of the file:
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@@
   (symbol (lib_id "Memory_Flash:W25Q128JVS") (at 229.87 69.85 0) (unit 1)
     (in_bom yes) (on_board yes) (dnp no)
-    (property "Reference" "U7" (at 214.63 79.375 0)
+    (property "Reference" "U7" (at 212.725 79.375 0)
       (effects (font (size 1.27 1.27)) (justify left))
     )
-    (property "Value" "W25Q128JVSIQ" (at 214.63 81.915 0)
+    (property "Value" "W25Q128JVSIQ" (at 212.725 81.915 0)
       (effects (font (size 1.27 1.27)) (justify left))
     )

Commit message: Add files via upload
Connections:
- net INT3: now also U4.50 (PA15); no longer U4.54 (PD2)
Changed lines of the file:
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@@
   (no_connect (at 219.71 74.93))
   (no_connect (at 117.475 133.985))
-  (no_connect (at 117.475 123.825))
   (no_connect (at 117.475 149.225))
   (no_connect (at 81.915 108.585))
@@
   (no_connect (at 117.475 141.605))
   (no_connect (at 117.475 139.065))
+  (no_connect (at 81.915 103.505))
   (no_connect (at 117.475 151.765))
   (wire (pts (xy 46.99 154.94) (xy 44.45 154.94))
@@
     )
   )
-  (global_label "INT3" (shape input) (at 81.915 103.505 180) (fields_autoplaced)
-    (effects (font (size 1.27 1.27)) (justify right))
-    (property "Intersheetrefs" "${INTERSHEET_REFS}" (at 74.8968 103.505 0)
-      (effects (font (size 1.27 1.27)) (justify right) hide)
-    )
-  )
+  (global_label "INT3" (shape input) (at 117.475 123.825 0) (fields_autoplaced)
+    (effects (font (size 1.27 1.27)) (justify left))
+    (property "Intersheetrefs" "${INTERSHEET_REFS}" (at 124.4932 123.825 0)
+      (effects (font (size 1.27 1.27)) (justify left) hide)
+    )
+  )

Commit message: Add files via upload
Connections:
- net CS_EXTRA: now also U4.41 (PA8); no longer U4.40 (PC9)
- net ESC: now also U4.38 (PC7); no longer U4.37 (PC6)
- net FLASH_CS: now also U4.40 (PC9); no longer U4.39 (PC8)
- net INT_GPS: now also U4.39 (PC8); no longer U4.38 (PC7)
- net Servo 2: now also U4.34 (PB13); no longer U4.33 (PB12)
- net Servo 3: now also U4.35 (PB14); no longer U4.34 (PB13)
- net Servo 4: now also U4.36 (PB15); no longer U4.35 (PB14)
- net Servo 5: now also U4.37 (PC6); no longer U4.36 (PB15)

Commit message: Add files via upload
Connections:
- net INT_GPS: no longer names the net of U4.39 (PC8)
- no-connect marks 12 -> 13
Changed lines of the file:
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@@
   (no_connect (at 219.71 72.39))
   (no_connect (at 219.71 74.93))
+  (no_connect (at 81.915 128.905))
   (no_connect (at 117.475 133.985))
   (no_connect (at 117.475 149.225))
@@
       (effects (font (size 1.27 1.27)) (justify right) hide)
     )
-  )
-  (global_label "INT_GPS" (shape input) (at 81.915 128.905 180) (fields_autoplaced)
-    (effects (font (size 1.27 1.27)) (justify right))
-    (property "Intersheetrefs" "${INTERSHEET_REFS}" (at 71.3892 128.905 0)
-      (effects (font (size 1.27 1.27)) (justify right) hide)
-    )

Commit message: Add files via upload
Parts:
- added D1: GREEN, LED_SMD:LED_0603_1608Metric, symbol Device:LED
- added R9: 1k, Resistor_SMD:R_0603_1608Metric, symbol Device:R
- D1: value RED -> GREEN
Connections:
- net GND: now also R9.2
- net LED3: now reaches U4.39 (PC8)
- net LED3: now also D1.2 (A)
- new net: D1.1 (K), R9.1
- no-connect marks 13 -> 12
Other:
- moved on the sheet: D1, R9
Changed lines of the file:
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@@
   (no_connect (at 219.71 72.39))
   (no_connect (at 219.71 74.93))
-  (no_connect (at 81.915 128.905))
   (no_connect (at 117.475 133.985))
   (no_connect (at 117.475 149.225))
@@
     (stroke (width 0) (type default))
   )
-  (wire (pts (xy 149.86 93.345) (xy 147.32 93.345))
+  (wire (pts (xy 148.59 80.645) (xy 146.05 80.645))
     (stroke (width 0) (type default))
   )
@@
     (stroke (width 0) (type default))
   )
-  (wire (pts (xy 147.32 93.345) (xy 147.32 95.885))
+  (wire (pts (xy 146.05 80.645) (xy 146.05 83.185))
     (stroke (width 0) (type default))
   )
@@
     (stroke (width 0) (type default))
   )
+  (wire (pts (xy 144.78 158.75) (xy 144.78 161.29))
+    (stroke (width 0) (type default))
+  )
   (wire (pts (xy 210.82 60.96) (xy 210.82 62.23))
     (stroke (width 0) (type default))
@@
   )
   (wire (pts (xy 52.07 120.65) (xy 52.07 120.015))
+    (stroke (width 0) (type default))
+  )
+  (wire (pts (xy 147.32 158.75) (xy 144.78 158.75))
     (stroke (width 0) (type default))
   )
@@
     )
   )
+  (global_label "LED3" (shape input) (at 147.32 158.75 0)
+    (effects (font (size 1.27 1.27)) (justify left))
+    (property "Intersheetrefs" "${INTERSHEET_REFS}" (at 147.32 158.75 0)
+      (effects (font (size 1.27 1.27)) hide)
+    )
+  )
   (global_label "INT_PI" (shape input) (at 81.915 144.145 180) (fields_autoplaced)
     (effects (font (size 1.27 1.27)) (justify right))
@@
     )
   )
-  (global_label "LED1" (shape input) (at 149.86 93.345 0)
-    (effects (font (size 1.27 1.27)) (justify left))
-    (property "Intersheetrefs" "${INTERSHEET_REFS}" (at 149.86 93.345 0)
+  (global_label "LED1" (shape input) (at 148.59 80.645 0)
+    (effects (font (size 1.27 1.27)) (justify left))
+    (property "Intersheetrefs" "${INTERSHEET_REFS}" (at 148.59 80.645 0)
+      (effects (font (size 1.27 1.27)) hide)
+    )
+  )
+  (global_label "LED3" (shape input) (at 81.915 128.905 180)
+    (effects (font (size 1.27 1.27)) (justify right))
+    (property "Intersheetrefs" "${INTERSHEET_REFS}" (at 81.915 128.905 0)
       (effects (font (size 1.27 1.27)) hide)
     )
@@
     )
   )
-  (symbol (lib_id "Device:LED") (at 147.32 99.695 90) (unit 1)
-    (in_bom yes) (on_board yes) (dnp no)
-    (property "Reference" "D1" (at 142.875 99.06 90)
-      (effects (font (size 1.27 1.27)))
-    )
-    (property "Value" "RED" (at 142.875 101.6 90)
-      (effects (font (size 1.27 1.27)))
-    )
-    (property "Footprint" "LED_SMD:LED_0603_1608Metric" (at 147.32 99.695 0)
-      (effects (font (size 1.27 1.27)) hide)
-    )
-    (property "Datasheet" "~" (at 147.32 99.695 0)
+  (symbol (lib_id "Device:LED") (at 146.05 86.995 90) (unit 1)
+    (in_bom yes) (on_board yes) (dnp no)
+    (property "Reference" "D1" (at 141.605 86.36 90)
+      (effects (font (size 1.27 1.27)))
+    )
+    (property "Value" "GREEN" (at 141.605 88.9 90)
+      (effects (font (size 1.27 1.27)))
+    )
+    (property "Footprint" "LED_SMD:LED_0603_1608Metric" (at 146.05 86.995 0)
+      (effects (font (size 1.27 1.27)) hide)
+    )
+    (property "Datasheet" "~" (at 146.05 86.995 0)
       (effects (font (size 1.27 1.27)) hide)
     )
@@
       (effects (font (size 1.27 1.27)))
     )
-    (property "Value" "RED" (at 40.005 163.195 90)
+    (property "Value" "GREEN" (at 40.005 163.195 90)
       (effects (font (size 1.27 1.27)))
     )
@@
         (path "/619b7a98-ea9e-4ba1-a6ac-2aefa32bb41a/ba9d85a1-a354-40b5-8abd-109371bb61fa"
           (reference "Y1") (unit 1)
+        )
+      )
+    )
+  )
+  (symbol (lib_id "Device:LED") (at 144.78 165.1 90) (unit 1)
+    (in_bom yes) (on_board yes) (dnp no)
+    (property "Reference" "D1" (at 140.335 164.465 90)
+      (effects (font (size 1.27 1.27)))
+    )
+    (property "Value" "GREEN" (at 140.335 167.005 90)
+      (effects (font (size 1.27 1.27)))
+    )
+    (property "Footprint" "LED_SMD:LED_0603_1608Metric" (at 144.78 165.1 0)
+      (effects (font (size 1.27 1.27)) hide)
+    )
+    (property "Datasheet" "~" (at 144.78 165.1 0)
+      (effects (font (size 1.27 1.27)) hide)
+    )
+    (pin "1")
+    (pin "2")
+    (instances
+      (project "FlightComputer"
+        (path "/619b7a98-ea9e-4ba1-a6ac-2aefa32bb41a"
+          (reference "D1") (unit 1)
+        )
+        (path "/619b7a98-ea9e-4ba1-a6ac-2aefa32bb41a/860700d0-b412-4191-a92c-98767c85d1ad"
+          (reference "D1") (unit 1)
+        )
+        (path "/619b7a98-ea9e-4ba1-a6ac-2aefa32bb41a/ba9d85a1-a354-40b5-8abd-109371bb61fa"
+          (reference "D9") (unit 1)
         )
       )
@@
     )
   )
-  (symbol (lib_id "power:GND") (at 147.32 111.125 0) (unit 1)
-    (in_bom yes) (on_board yes) (dnp no)
-    (property "Reference" "#PWR041" (at 147.32 117.475 0)
-      (effects (font (size 1.27 1.27)) hide)
-    )
-    (property "Value" "GND" (at 147.32 114.935 0)
-      (effects (font (size 1.27 1.27)))
-    )
-    (property "Footprint" "" (at 147.32 111.125 0)
-      (effects (font (size 1.27 1.27)) hide)
-    )
-    (property "Datasheet" "" (at 147.32 111.125 0)
+  (symbol (lib_id "power:GND") (at 146.05 98.425 0) (unit 1)
+    (in_bom yes) (on_board yes) (dnp no)
+    (property "Reference" "#PWR041" (at 146.05 104.775 0)
+      (effects (font (size 1.27 1.27)) hide)
+    )
+    (property "Value" "GND" (at 146.05 102.235 0)
+      (effects (font (size 1.27 1.27)))
+    )
+    (property "Footprint" "" (at 146.05 98.425 0)
+      (effects (font (size 1.27 1.27)) hide)
+    )
+    (property "Datasheet" "" (at 146.05 98.425 0)
       (effects (font (size 1.27 1.27)) hide)
     )
@@
         (path "/619b7a98-ea9e-4ba1-a6ac-2aefa32bb41a/ba9d85a1-a354-40b5-8abd-109371bb61fa"
           (reference "C25") (unit 1)
+        )
+      )
+    )
+  )
+  (symbol (lib_id "Device:R") (at 144.78 172.72 0) (mirror y) (unit 1)
+    (in_bom yes) (on_board yes) (dnp no)
+    (property "Reference" "R9" (at 142.875 171.577 0)
+      (effects (font (size 1.27 1.27)) (justify left))
+    )
+    (property "Value" "1k" (at 142.875 174.117 0)
+      (effects (font (size 1.27 1.27)) (justify left))
+    )
+    (property "Footprint" "Resistor_SMD:R_0603_1608Metric" (at 146.558 172.72 90)
+      (effects (font (size 1.27 1.27)) hide)
+    )
+    (property "Datasheet" "~" (at 144.78 172.72 0)
+      (effects (font (size 1.27 1.27)) hide)
+    )
+    (pin "1")
+    (pin "2")
+    (instances
+      (project "FCRev2"
+        (path "/4bfaf9f4-833d-4b89-870a-6e523da66099"
+          (reference "R9") (unit 1)
+        )
+      )
+      (project "FlightComputer"
+        (path "/619b7a98-ea9e-4ba1-a6ac-2aefa32bb41a"
+          (reference "R7") (unit 1)
+        )
+        (path "/619b7a98-ea9e-4ba1-a6ac-2aefa32bb41a/860700d0-b412-4191-a92c-98767c85d1ad"
+          (reference "R2") (unit 1)
+        )
+        (path "/619b7a98-ea9e-4ba1-a6ac-2aefa32bb41a/234b6c4f-327d-42b9-b59c-801877bb3b05"
+          (reference "R12") (unit 1)
+        )
+        (path "/619b7a98-ea9e-4ba1-a6ac-2aefa32bb41a/ba9d85a1-a354-40b5-8abd-109371bb61fa"
+          (reference "R25") (unit 1)
+        )
+      )
+      (project "FlightComputer"
+        (path "/bd2ca0f3-16be-405d-8265-527d0a4fe5c7"
+          (reference "R17") (unit 1)
         )
       )
@@
     )
   )
-  (symbol (lib_id "Device:R") (at 147.32 107.315 0) (mirror y) (unit 1)
-    (in_bom yes) (on_board yes) (dnp no)
-    (property "Reference" "R9" (at 145.415 106.172 0)
-      (effects (font (size 1.27 1.27)) (justify left))
-    )
-    (property "Value" "1k" (at 145.415 108.712 0)
-      (effects (font (size 1.27 1.27)) (justify left))
-    )
-    (property "Footprint" "Resistor_SMD:R_0603_1608Metric" (at 149.098 107.315 90)
-      (effects (font (size 1.27 1.27)) hide)
-    )
-    (property "Datasheet" "~" (at 147.32 107.315 0)
+  (symbol (lib_id "Device:R") (at 146.05 94.615 0) (mirror y) (unit 1)
+    (in_bom yes) (on_board yes) (dnp no)
+    (property "Reference" "R9" (at 144.145 93.472 0)
+      (effects (font (size 1.27 1.27)) (justify left))
+    )
+    (property "Value" "1k" (at 144.145 96.012 0)
+      (effects (font (size 1.27 1.27)) (justify left))
+    )
+    (property "Footprint" "Resistor_SMD:R_0603_1608Metric" (at 147.828 94.615 90)
+      (effects (font (size 1.27 1.27)) hide)
+    )
+    (property "Datasheet" "~" (at 146.05 94.615 0)
       (effects (font (size 1.27 1.27)) hide)
     )
@@
         )
       )
+    )
+  )
+  (symbol (lib_id "power:GND") (at 144.78 176.53 0) (unit 1)
+    (in_bom yes) (on_board yes) (dnp no)
+    (property "Reference" "#PWR041" (at 144.78 182.88 0)
+      (effects (font (size 1.27 1.27)) hide)
+    )
+    (property "Value" "GND" (at 144.78 180.34 0)
+      (effects (font (size 1.27 1.27)))
+    )
+    (property "Footprint" "" (at 144.78 176.53 0)
+      (effects (font (size 1.27 1.27)) hide)
+    )
+    (property "Datasheet" "" (at 144.78 176.53 0)
+      (effects (font (size 1.27 1.27)) hide)
+    )
+    (pin "1")
+    (instances
+      (project "STM32F4_REV2"
+        (path "/58802e77-440d-4789-b1be-932d1522915a"
+          (reference "#PWR041") (unit 1)
+        )
+      )
+      (project "FlightComputer"
+        (path "/619b7a98-ea9e-4ba1-a6ac-2aefa32bb41a"
+          (reference "#PWR083") (unit 1)
+        )
+        (path "/619b7a98-ea9e-4ba1-a6ac-2aefa32bb41a/ba9d85a1-a354-40b5-8abd-109371bb61fa"
+          (reference "#PWR064") (unit 1)
+        )
+      )

Commit message: Add files via upload
Other:
- note added: "LEDs"
- note added: "RELEASE: HIGH PRESS: LOW"
- note added: "Section 6.3.18: NRST pin is connected to an internal pull-up resistor. User must ensure level on NRST pin can go below VIL(NRST) max level specified in Table 59. Otherwise reset is not taken into account by device."
- note added: "TIM1_CH1N"
- note added: "TIM1_CH2N"
- note added: "TIM1_CH3N"
- note added: "TIM2_CH2"
- note added: "TIM2_CH3"
- note added: "TIM3_CH1"
- note added: "Table 18: Capacitance of external capacitor with a single VCAP pin avaliable should be 4.7uF"
- note removed: "RELEASE: FLOATING PRESS: GND"
- moved on the sheet: C20, D1, R1, R8, R9, SW1, U7
