File: Microcontroller.kicad_sch (KiCad schematic)
At the start: 33 parts, among them SW1 KMR221GLFS, U4 STM32F446RET6, U7 W25Q128JVSIQ, Y1 16MHz

Commit message: Add files via upload
Connections:
- net INT_MAG: now reaches U4.33 (PB12)
- no-connect marks 12 -> 11
Other:
- note added: "ADC12_IN4"
- note added: "I2C1_SCL"
- note added: "I2C1_SDA"
- note added: "SPI1_MISO"
- note added: "SPI1_MOSI"
- note added: "SPI1_SCK"
- moved on the sheet: R12, R13
