File: Power.kicad_sch (KiCad schematic)
At the start: 34 parts, among them IC1 LMR33640DDDAR, J13 SM02B-GHS-TB, J16 SM02B-GHS-TB, J17 Screw_Terminal_01x02, Q1 SI2369BDS-T1-GE3 30V 5.6A, U3 AP7361C-33ER-13

Commit message: Add files via upload
Parts:
- added D36 (x2): PESD5V0U1UA, Diode_SMD:D_SOD-323, symbol Device:D
Connections:
- net GND: now also D36.2 (A), D36.2 (A)
- net at F9.2, J13.1 (Pin_1): now also D36.1 (K)
- net at F8.2, J16.1 (Pin_1): now also D36.1 (K)
Changed lines of the file:
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@@
   (junction (at 192.405 49.53) (diameter 0) (color 0 0 0 0)
   )
+  (junction (at 236.855 122.555) (diameter 0) (color 0 0 0 0)
+  )
   (junction (at 125.095 59.69) (diameter 0) (color 0 0 0 0)
   )
@@
   )
   (junction (at 203.835 59.69) (diameter 0) (color 0 0 0 0)
+  )
+  (junction (at 239.395 142.875) (diameter 0) (color 0 0 0 0)
+  )
+  (junction (at 243.205 150.495) (diameter 0) (color 0 0 0 0)
+  )
+  (junction (at 242.57 130.175) (diameter 0) (color 0 0 0 0)
   )
   (junction (at 248.285 49.53) (diameter 0) (color 0 0 0 0)
@@
     (stroke (width 0) (type default))
   )
-  (wire (pts (xy 234.95 142.875) (xy 243.205 142.875))
+  (wire (pts (xy 234.95 142.875) (xy 239.395 142.875))
     (stroke (width 0) (type default))
   )
@@
     (stroke (width 0) (type default))
   )
+  (wire (pts (xy 236.855 130.175) (xy 242.57 130.175))
+    (stroke (width 0) (type default))
+  )
   (wire (pts (xy 203.835 49.53) (xy 201.93 49.53))
     (stroke (width 0) (type default))
   )
+  (wire (pts (xy 242.57 130.175) (xy 242.57 125.095))
+    (stroke (width 0) (type default))
+  )
   (wire (pts (xy 114.3 146.05) (xy 125.095 146.05))
     (stroke (width 0) (type default))
@@
     (stroke (width 0) (type default))
   )
+  (wire (pts (xy 243.205 150.495) (xy 243.205 145.415))
+    (stroke (width 0) (type default))
+  )
   (wire (pts (xy 136.525 50.8) (xy 136.525 49.53))
     (stroke (width 0) (type default))
@@
     (stroke (width 0) (type default))
   )
+  (wire (pts (xy 239.395 150.495) (xy 243.205 150.495))
+    (stroke (width 0) (type default))
+  )
   (wire (pts (xy 59.69 54.61) (xy 62.23 54.61))
     (stroke (width 0) (type default))
@@
     (stroke (width 0) (type default))
   )
+  (wire (pts (xy 239.395 142.875) (xy 243.205 142.875))
+    (stroke (width 0) (type default))
+  )
   (wire (pts (xy 236.855 59.69) (xy 225.425 59.69))
     (stroke (width 0) (type default))
@@
     (stroke (width 0) (type default))
   )
-  (wire (pts (xy 235.585 122.555) (xy 242.57 122.555))
+  (wire (pts (xy 235.585 122.555) (xy 236.855 122.555))
     (stroke (width 0) (type default))
   )
@@
   )
   (wire (pts (xy 67.31 62.23) (xy 74.93 62.23))
+    (stroke (width 0) (type default))
+  )
+  (wire (pts (xy 236.855 122.555) (xy 242.57 122.555))
     (stroke (width 0) (type default))
   )
@@
     )
   )
-  (symbol (lib_id "power:GND") (at 243.205 145.415 0) (unit 1)
-    (in_bom yes) (on_board yes) (dnp no) (fields_autoplaced)
-    (property "Reference" "#PWR035" (at 243.205 151.765 0)
-      (effects (font (size 1.27 1.27)) hide)
-    )
-    (property "Value" "GND" (at 243.205 150.495 0)
-      (effects (font (size 1.27 1.27)))
-    )
-    (property "Footprint" "" (at 243.205 145.415 0)
-      (effects (font (size 1.27 1.27)) hide)
-    )
-    (property "Datasheet" "" (at 243.205 145.415 0)
+  (symbol (lib_id "power:GND") (at 243.205 150.495 0) (unit 1)
+    (in_bom yes) (on_board yes) (dnp no) (fields_autoplaced)
+    (property "Reference" "#PWR035" (at 243.205 156.845 0)
+      (effects (font (size 1.27 1.27)) hide)
+    )
+    (property "Value" "GND" (at 243.205 155.575 0)
+      (effects (font (size 1.27 1.27)))
+    )
+    (property "Footprint" "" (at 243.205 150.495 0)
+      (effects (font (size 1.27 1.27)) hide)
+    )
+    (property "Datasheet" "" (at 243.205 150.495 0)
       (effects (font (size 1.27 1.27)) hide)
     )
@@
         (path "/619b7a98-ea9e-4ba1-a6ac-2aefa32bb41a/234b6c4f-327d-42b9-b59c-801877bb3b05"
           (reference "#PWR056") (unit 1)
+        )
+      )
+    )
+  )
+  (symbol (lib_id "Device:D") (at 236.855 126.365 270) (unit 1)
+    (in_bom yes) (on_board yes) (dnp no)
+    (property "Reference" "D36" (at 230.505 127 90)
+      (effects (font (size 1.27 1.27)) (justify left))
+    )
+    (property "Value" "PESD5V0U1UA" (at 218.44 129.54 90)
+      (effects (font (size 1.27 1.27)) (justify left))
+    )
+    (property "Footprint" "Diode_SMD:D_SOD-323" (at 236.855 126.365 0)
+      (effects (font (size 1.27 1.27)) hide)
+    )
+    (property "Datasheet" "~" (at 236.855 126.365 0)
+      (effects (font (size 1.27 1.27)) hide)
+    )
+    (property "Sim.Device" "D" (at 236.855 126.365 0)
+      (effects (font (size 1.27 1.27)) hide)
+    )
+    (property "Sim.Pins" "1=K 2=A" (at 236.855 126.365 0)
+      (effects (font (size 1.27 1.27)) hide)
+    )
+    (pin "1")
+    (pin "2")
+    (instances
+      (project "FlightComputer"
+        (path "/619b7a98-ea9e-4ba1-a6ac-2aefa32bb41a/234b6c4f-327d-42b9-b59c-801877bb3b05"
+          (reference "D36") (unit 1)
+        )
+        (path "/619b7a98-ea9e-4ba1-a6ac-2aefa32bb41a/860700d0-b412-4191-a92c-98767c85d1ad"
+          (reference "D3") (unit 1)
         )
       )
@@
     )
   )
-  (symbol (lib_id "power:GND") (at 242.57 125.095 0) (unit 1)
-    (in_bom yes) (on_board yes) (dnp no) (fields_autoplaced)
-    (property "Reference" "#PWR042" (at 242.57 131.445 0)
-      (effects (font (size 1.27 1.27)) hide)
-    )
-    (property "Value" "GND" (at 242.57 130.175 0)
-      (effects (font (size 1.27 1.27)))
-    )
-    (property "Footprint" "" (at 242.57 125.095 0)
-      (effects (font (size 1.27 1.27)) hide)
-    )
-    (property "Datasheet" "" (at 242.57 125.095 0)
+  (symbol (lib_id "power:GND") (at 242.57 130.175 0) (unit 1)
+    (in_bom yes) (on_board yes) (dnp no) (fields_autoplaced)
+    (property "Reference" "#PWR042" (at 242.57 136.525 0)
+      (effects (font (size 1.27 1.27)) hide)
+    )
+    (property "Value" "GND" (at 242.57 135.255 0)
+      (effects (font (size 1.27 1.27)))
+    )
+    (property "Footprint" "" (at 242.57 130.175 0)
+      (effects (font (size 1.27 1.27)) hide)
+    )
+    (property "Datasheet" "" (at 242.57 130.175 0)
       (effects (font (size 1.27 1.27)) hide)
     )
@@
         )
       )
+    )
+  )
+  (symbol (lib_id "Device:D") (at 239.395 146.685 270) (unit 1)
+    (in_bom yes) (on_board yes) (dnp no)
+    (property "Reference" "D36" (at 234.315 146.05 90)
+      (effects (font (size 1.27 1.27)) (justify left))
+    )
+    (property "Value" "PESD5V0U1UA" (at 222.25 148.59 90)
+      (effects (font (size 1.27 1.27)) (justify left))
+    )
+    (property "Footprint" "Diode_SMD:D_SOD-323" (at 239.395 146.685 0)
+      (effects (font (size 1.27 1.27)) hide)
+    )
+    (property "Datasheet" "~" (at 239.395 146.685 0)
+      (effects (font (size 1.27 1.27)) hide)
+    )
+    (property "Sim.Device" "D" (at 239.395 146.685 0)
+      (effects (font (size 1.27 1.27)) hide)
+    )
+    (property "Sim.Pins" "1=K 2=A" (at 239.395 146.685 0)
+      (effects (font (size 1.27 1.27)) hide)
+    )
+    (pin "1")
+    (pin "2")
+    (instances
+      (project "FlightComputer"
+        (path "/619b7a98-ea9e-4ba1-a6ac-2aefa32bb41a/234b6c4f-327d-42b9-b59c-801877bb3b05"
+          (reference "D36") (unit 1)
+        )
+        (path "/619b7a98-ea9e-4ba1-a6ac-2aefa32bb41a/860700d0-b412-4191-a92c-98767c85d1ad"
+          (reference "D4") (unit 1)
+        )
+      )

Commit message: Add files via upload
Other:
- moved on the sheet: C26, C27, D36, F8, F9, TP3, U3

Commit message: Add files via upload
Parts:
- D36: value PESD5V0U1UA -> TPESD5V0U1UA
Changed lines of the file:
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@@
       (effects (font (size 1.27 1.27)) (justify left))
     )
-    (property "Value" "PESD5V0U1UA" (at 219.71 129.54 90)
+    (property "Value" "TPESD5V0U1UA" (at 219.71 129.54 90)
       (effects (font (size 1.27 1.27)) (justify left))
     )
@@
       (effects (font (size 1.27 1.27)) (justify left))
     )
-    (property "Value" "PESD5V0U1UA" (at 222.25 148.59 90)
-      (effects (font (size 1.27 1.27)) (justify left))
-    )
+    (property "Value" "TPESD5V0U1UA" (at 222.25 148.59 90)
+      (effects (font (size 1.27 1.27)) (justify left))
+    )

Commit message: Add files via upload
Parts:
- D1: value GREEN -> RED
Other:
- moved on the sheet: C10, C11, C12, C14, C15, C16, C26, C27, C8, D1, D36, F8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

Commit message: Add files via upload
Other:
- note added: "INPUT: 6V - 26V Battery connects to a parallel XT60 connector with one port powering an electric fan and one port powering the PCB through the screw terminal (J2)"
- note removed: "INPUT: 6V - 26V Battery connects to a parallel XT60 connector with one port powering an electric fan and one port powering the PCB through the screw terminal"
- moved on the sheet: D36, F8, F9, J13

Commit message: Add files via upload
Changed lines of the file:
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@@
   (symbol (lib_id "Device:C") (at 187.325 53.34 90) (unit 1)
     (in_bom yes) (on_board yes) (dnp no)
-    (property "Reference" "C12" (at 193.04 54.61 90)
+    (property "Reference" "C12" (at 185.42 51.435 90)
       (effects (font (size 1.27 1.27)) (justify left))
     )
-    (property "Value" "0.1uF" (at 194.31 57.15 90)
+    (property "Value" "0.1uF" (at 185.42 55.245 90)
       (effects (font (size 1.27 1.27)) (justify left))
     )
