File: Sensors.kicad_sch (KiCad schematic)
At the start: 16 parts, among them U1 LPS22HH, U5 BMI270, U6 LIS3MDL, U6 NEO-M9N

Commit message: Add files via upload
Parts:
- D13: value CESD3V3D3 YU -> PESD5V0U1UA
Other:
- note added: "Pin 1 or 10"
- note added: "Pin 4"
- note added: "Pin 5"
- note added: "Pin 6"
- note added: "Pin 8"
Changed lines of the file:
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@@
     (effects (font (size 3 3)) (justify left bottom))
+  )
+  (text "Pin 6" (at 43.815 130.81 0)
+    (effects (font (size 1.27 1.27)) (justify left bottom))
+  )
+  (text "Pin 4" (at 61.595 138.43 0)
+    (effects (font (size 1.27 1.27)) (justify left bottom))
+  )
+  (text "Pin 5" (at 33.02 130.81 0)
+    (effects (font (size 1.27 1.27)) (justify left bottom))
   )
   (text "I2C is fast enough for my application" (at 59.69 29.21 0)
     (effects (font (size 1.27 1.27)) (justify left bottom))
   )
+  (text "Pin 8" (at 43.815 69.215 0)
+    (effects (font (size 1.27 1.27)) (justify left bottom))
+  )
   (text "Inertial Measurement Unit" (at 23.495 38.1 0)
     (effects (font (size 3 3)) (justify left bottom))
@@
     (effects (font (size 3 3) (thickness 0.6) bold) (justify left bottom))
   )
+  (text "Pin 5" (at 31.115 69.215 0)
+    (effects (font (size 1.27 1.27)) (justify left bottom))
+  )
   (text "Barometric Pressure Sensor" (at 103.505 38.1 0)
     (effects (font (size 3 3)) (justify left bottom))
+  )
+  (text "Pin 1 or 10" (at 107.95 68.58 0)
+    (effects (font (size 1.27 1.27)) (justify left bottom))
   )
   (global_label "SDA" (shape input) (at 146.685 54.61 0) (fields_autoplaced)
@@
       (effects (font (size 1.27 1.27)))
     )
-    (property "Value" "CESD3V3D3 YU" (at 189.865 85.09 0)
-      (effects (font (size 1.27 1.27)))
-    )
+    (property "Value" "PESD5V0U1UA" (at 189.865 85.09 0)
+      (effects (font (size 1.27 1.27)))
+    )

Commit message: Add files via upload
Parts:
- D13: value PESD5V0U1UA -> TPESD5V0U1UA
Changed lines of the file:
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@@
       (effects (font (size 1.27 1.27)))
     )
-    (property "Value" "PESD5V0U1UA" (at 189.865 85.09 0)
+    (property "Value" "TPESD5V0U1UA" (at 189.865 85.09 0)
       (effects (font (size 1.27 1.27)))
     )

Commit message: Add files via upload
Other:
- note added: "uart has global interrupt. no need for interrupts for uarts"
Changed lines of the file:
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@@
+    (effects (font (size 1.27 1.27)) (justify left bottom))
+  )
+  (text "uart has global interrupt. no need for interrupts for uarts"
+    (at 203.835 42.545 0)
     (effects (font (size 1.27 1.27)) (justify left bottom))
   )

Commit message: Add files via upload
Connections:
- net INT_GPS: no longer names the net of U6.4 (EXTINT)
- no-connect marks 15 -> 16
Changed lines of the file:
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@@
   )
   (no_connect (at 201.295 92.71))
+  (no_connect (at 201.295 97.79))
   (no_connect (at 201.295 113.03))
   (no_connect (at 201.295 120.65))
@@
       (effects (font (size 1.27 1.27)) (justify right) hide)
     )
-  )
-  (global_label "INT_GPS" (shape input) (at 201.295 97.79 180) (fields_autoplaced)
-    (effects (font (size 1.27 1.27)) (justify right))
-    (property "Intersheetrefs" "${INTERSHEET_REFS}" (at 190.7692 97.79 0)
-      (effects (font (size 1.27 1.27)) (justify right) hide)
-    )

Commit message: Add files via upload
Parts:
- added TP3: TestPoint, TestPoint:TestPoint_Pad_D1.5mm, symbol Connector:TestPoint
Connections:
- net at U6.1 (SAFEBOOT_N): now also TP3.1
- no-connect marks 16 -> 15
Changed lines of the file:
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@@
   (junction (at 52.705 140.335) (diameter 0) (color 0 0 0 0)
   )
-  (no_connect (at 201.295 92.71))
   (no_connect (at 201.295 97.79))
   (no_connect (at 201.295 113.03))
@@
     (stroke (width 0) (type default))
   )
-  (wire (pts (xy 186.055 87.63) (xy 187.325 87.63))
+  (wire (pts (xy 178.435 87.63) (xy 187.325 87.63))
     (stroke (width 0) (type default))
   )
@@
     (stroke (width 0) (type default))
   )
-  (wire (pts (xy 197.485 95.25) (xy 201.295 95.25))
+  (wire (pts (xy 184.15 95.25) (xy 201.295 95.25))
     (stroke (width 0) (type default))
   )
@@
     (stroke (width 0) (type default))
   )
-  (wire (pts (xy 186.055 88.9) (xy 186.055 87.63))
+  (wire (pts (xy 178.435 88.9) (xy 178.435 87.63))
     (stroke (width 0) (type default))
   )
@@
     )
   )
-  (symbol (lib_id "power:+3V3") (at 197.485 95.25 0) (unit 1)
+  (symbol (lib_id "power:+3V3") (at 184.15 95.25 0) (unit 1)
     (in_bom yes) (on_board yes) (dnp no) (fields_autoplaced)
-    (property "Reference" "#PWR054" (at 197.485 99.06 0)
-      (effects (font (size 1.27 1.27)) hide)
-    )
-    (property "Value" "+3V3" (at 197.485 91.7956 0)
-      (effects (font (size 1.27 1.27)))
-    )
-    (property "Footprint" "" (at 197.485 95.25 0)
-      (effects (font (size 1.27 1.27)) hide)
-    )
-    (property "Datasheet" "" (at 197.485 95.25 0)
+    (property "Reference" "#PWR054" (at 184.15 99.06 0)
+      (effects (font (size 1.27 1.27)) hide)
+    )
+    (property "Value" "+3V3" (at 184.15 91.7956 0)
+      (effects (font (size 1.27 1.27)))
+    )
+    (property "Footprint" "" (at 184.15 95.25 0)
+      (effects (font (size 1.27 1.27)) hide)
+    )
+    (property "Datasheet" "" (at 184.15 95.25 0)
       (effects (font (size 1.27 1.27)) hide)
     )
@@
     )
   )
-  (symbol (lib_id "power:GND") (at 186.055 88.9 0) (unit 1)
-    (in_bom yes) (on_board yes) (dnp no)
-    (property "Reference" "#PWR023" (at 186.055 95.25 0)
-      (effects (font (size 1.27 1.27)) hide)
-    )
-    (property "Value" "GND" (at 186.055 92.71 0)
-      (effects (font (size 1.27 1.27)))
-    )
-    (property "Footprint" "" (at 186.055 88.9 0)
-      (effects (font (size 1.27 1.27)) hide)
-    )
-    (property "Datasheet" "" (at 186.055 88.9 0)
+  (symbol (lib_id "power:GND") (at 178.435 88.9 0) (unit 1)
+    (in_bom yes) (on_board yes) (dnp no)
+    (property "Reference" "#PWR023" (at 178.435 95.25 0)
+      (effects (font (size 1.27 1.27)) hide)
+    )
+    (property "Value" "GND" (at 178.435 92.71 0)
+      (effects (font (size 1.27 1.27)))
+    )
+    (property "Footprint" "" (at 178.435 88.9 0)
+      (effects (font (size 1.27 1.27)) hide)
+    )
+    (property "Datasheet" "" (at 178.435 88.9 0)
       (effects (font (size 1.27 1.27)) hide)
     )
@@
         )
       )
+    )
+  )
+  (symbol (lib_id "Connector:TestPoint") (at 201.295 92.71 90) (unit 1)
+    (in_bom yes) (on_board yes) (dnp no)
+    (property "Reference" "TP3" (at 196.85 93.98 90)
+      (effects (font (size 1.27 1.27)) (justify left))
+    )
+    (property "Value" "TestPoint" (at 196.85 91.44 90)
+      (effects (font (size 1.27 1.27)) (justify left))
+    )
+    (property "Footprint" "TestPoint:TestPoint_Pad_D1.5mm" (at 201.295 87.63 0)
+      (effects (font (size 1.27 1.27)) hide)
+    )
+    (property "Datasheet" "~" (at 201.295 87.63 0)
+      (effects (font (size 1.27 1.27)) hide)
+    )
+    (pin "1")
+    (instances
+      (project "FlightComputer"
+        (path "/619b7a98-ea9e-4ba1-a6ac-2aefa32bb41a"
+          (reference "TP3") (unit 1)
+        )
+        (path "/619b7a98-ea9e-4ba1-a6ac-2aefa32bb41a/860700d0-b412-4191-a92c-98767c85d1ad"
+          (reference "TP4") (unit 1)
+        )
+        (path "/619b7a98-ea9e-4ba1-a6ac-2aefa32bb41a/14b26996-81b8-4501-80f0-d5b7670415f0"
+          (reference "TP6") (unit 1)
+        )
+      )

Commit message: Add files via upload
Parts:
- removed TP3: TestPoint, TestPoint:TestPoint_Pad_D1.5mm, symbol Connector:TestPoint
- added TP4: TestPoint, TestPoint:TestPoint_Keystone_5000-5004_Miniature, symbol Connector:TestPoint
Connections:
- net INT_MAG: now reaches U6.8 (DRDY)
- net at U6.1 (SAFEBOOT_N): now also TP4.1
- no-connect marks 15 -> 14
Other:
- note added: "13.75mil trace for 50 ohm impedance with JLC04161H-7628 stackup https://jlcpcb.com/pcb-impedance-calculator/"
- note added: "UART has global interrupt. No need for dedicated interrupt pins."
- note removed: "11.55mil trace for 50 ohm impedance with JLC7628 stackup https://cart.jlcpcb.com/impedanceCalculation"
- note removed: "uart has global interrupt. no need for interrupts for uarts"
- moved on the sheet: AE1, C28, C3, D13, L3, R14, U6
